File: KiCad/Weapon/Weapon.sch (KiCad schematic (older format))
At the start: 16 parts, among them IC1 ATMEGA328-P, P1 ICSP, P2 USB-TTL, Q1 NPN, U1 RFID-RC522, X1 16MHz

Commit message: Weapon Schematic Ready
Parts:
- removed C1, C2: 0.1uF, ~, symbol C
- removed C3, C4: 22pF, ~, symbol C
- removed D1, D2: LED, ~, symbol LED
- removed IC1: ATMEGA328-P, DIL28, symbol ATMEGA328-P
- removed P1: ICSP, symbol CONN_3X2
- removed P2: USB-TTL, symbol CONN_6
- removed Q1: NPN, ~, symbol NPN
- removed R1: 1k, ~, symbol R
- removed R2: 10k, ~, symbol R
- removed R3: 560, ~, symbol R
- removed R4: 330, ~, symbol R
- removed U1: RFID-RC522, symbol RFID-RC522
- removed X1: 16MHz, ~, symbol CRYSTAL
- added C? (x2): 22pF, ~, symbol C
- added C? (x2): 0.1uF, ~, symbol C
- added C? (x2): 4.7uF, ~, symbol C
- added C?: 100uF, ~, symbol C
- added D? (x2): LED, ~, symbol LED
- added D?: RED, ~, symbol LED
- added IC?: ATMEGA328-P, DIL28, symbol ATMEGA328-P
- added J?: MICRO_USB, symbol MICRO_USB
- added P?: USB-TTL, symbol CONN_6
- added P?: 2P_CGRID_M, symbol 2P_CGRID_M
- added P?: 2P_CGRID_M, ~, symbol 2P_CGRID_M
- added Q?: NPN, ~, symbol NPN
- added R? (x4): 10k, ~, symbol R
- added R?: 560, ~, symbol R
- added R? (x2): 330, ~, symbol R
- added R?: 2k, ~, symbol R
- added R?: 1k, ~, symbol R
- added U?: RFID-RC522, symbol RFID-RC522
- added U?: MCP73831, symbol MCP73831
- added U?: LM1084IT-3.3/NOPB, TO-220, symbol LM1084IT-3.3/NOPB
- added X?: 16MHz, ~, symbol CRYSTAL
Connections:
- net labels added: StatusLED, Trigger, VoltageSense
- wire segments 57 -> 81
Other:
- note added: "3.3 V Regulator\n"
- note added: "IR-LED Driver\n"
- note added: "MicroController\n"
- note added: "Programming Port"
- note added: "RFID Reader\n"
- note added: "Status LED\n"
- note added: "Trigger Conector\n"
- note added: "USB Lipo Charger\n"

Commit message: 3/19 Progress
KiCad - weapon component to module selection and pcb file created.

All schematic components on net and allocated
Parts:
- gave numbers to parts that had none: 29

Commit message: Revert "Revert "3/29 KiCad Updates""
This reverts commit 46467126b97e8d3ee2ff82587e11af580e6d6854.
Parts:
- added LS1: BUZZER, symbol BUZZER
- added Q1: NPN, ~, symbol NPN
- added R3: 560, ~, symbol R
- added R7: 330, ~, symbol R
- added S1: SLIDESWITCH, symbol SLIDESWITCH
- renumbered Q1 to Q2, R8 to R10, R9 to R11, R3 to R4, R4 to R5, R5 to R6, R6 to R8, R7 to R9
Connections:
- net GND: now also C3.2, R2.2, U1.2 (VSS), LS1.2 (Vout)
- net V-Bat: now also Q1.3 (C), S1.2 (Vout); no longer P1.2 (VCC)
- net StatusLED renamed LED/Buzzer
- net LED/Buzzer: now also R3.2
- new net: P1.2 (VCC), S1.1 (Vin)
- new net: Q1.1 (E), R7.1
- new net: Q1.2 (B), R3.1
- new net: LS1.1 (Vin), R7.2
Other:
- note added: "Shot Confirmation LED/Buzzer"
- note removed: "Status LED\n"
- moved on the sheet: D2, R6

Commit message: Revert "3/29 KiCad Updates"
This reverts commit a2529da1b40b1f6e0e832ed1976ed3be41434859.
Parts:
- removed LS1: BUZZER, symbol BUZZER
- removed Q1: NPN, ~, symbol NPN
- removed R3: 560, ~, symbol R
- removed R7: 330, ~, symbol R
- removed S1: SLIDESWITCH, symbol SLIDESWITCH
- renumbered Q2 to Q1, R4 to R3, R5 to R4, R6 to R5, R8 to R6, R9 to R7, R10 to R8, R11 to R9
Connections:
- net GND: no longer C3.2, R2.2, U1.2 (VSS)
- net V-Bat: now also P1.2 (VCC)
- net LED/Buzzer renamed StatusLED
Other:
- note added: "Status LED\n"
- note removed: "Shot Confirmation LED/Buzzer"
- moved on the sheet: D2, R5
