File: KiCad/Weapon/Weapon.sch (KiCad schematic (older format))
At the start: 34 parts, among them IC1 ATMEGA328-P, J1 MICRO_USB, P1 2P_CGRID_M, P2 USB-TTL, P3 2P_CGRID_M, Q1 NPN, Q2 NPN, U1 MCP73831, U2 RFID-RC522, U3 LM1084IT-3.3/NOPB, X1 16MHz

Commit message: Quick Update #1 4/16
Parts:
- removed R7: 330, ~, symbol R
Connections:
- net at Q1.1 (E): now also LS1.1 (Vin)
Changed lines of the file:
@@
 Sheet 1 1
 Title ""
-Date "23 mar 2015"
+Date "17 apr 2015"
 Rev ""
 Comp ""
@@
 Text GLabel 7400 1050 2    60   Input ~ 0
 V-Bat
-$Comp
-L R R7
-U 1 1 550F98A8
-P 7150 1450
-F 0 "R7" V 7230 1450 40  0000 C CNN
-F 1 "330" V 7157 1451 40  0000 C CNN
-F 2 "~" V 7080 1450 30  0000 C CNN
-F 3 "~" H 7150 1450 30  0000 C CNN
-	1    7150 1450
-	0    -1   -1   0
-$EndComp
 Wire Wire Line
 	6400 900  6400 850
@@
 Wire Wire Line
 	4050 6100 4000 6100
+Wire Wire Line
+	7400 1450 6900 1450
 $EndSCHEMATC
