File: KiCad/Weapon/Weapon.sch (KiCad schematic (older format))
At the start: 33 parts, among them IC1 ATMEGA328-P, J1 MICRO_USB, P1 2P_CGRID_M, P2 USB-TTL, P3 2P_CGRID_M, Q1 NPN, Q2 NPN, U1 MCP73831, U2 RFID-RC522, U3 LM1084IT-3.3/NOPB, X1 16MHz

Commit message: Quick Update #1 4/28
Added resistor (220) to buzzer in weapon sch,net,pcb
Parts:
- added R7: 220, ~, symbol R
Connections:
- net at Q1.1 (E): now also R7.1; no longer LS1.1 (Vin)
- new net: LS1.1 (Vin), R7.2
Changed lines of the file:
@@
 Sheet 1 1
 Title ""
-Date "17 apr 2015"
+Date "29 apr 2015"
 Rev ""
 Comp ""
@@
 Wire Wire Line
 	4050 6100 4000 6100
-Wire Wire Line
-	7400 1450 6900 1450
+$Comp
+L R R7
+U 1 1 55402F27
+P 7150 1450
+F 0 "R7" V 7230 1450 40  0000 C CNN
+F 1 "220" V 7157 1451 40  0000 C CNN
+F 2 "~" V 7080 1450 30  0000 C CNN
+F 3 "~" H 7150 1450 30  0000 C CNN
+	1    7150 1450
+	0    -1   -1   0
+$EndComp
 $EndSCHEMATC
