File: KiCad/Weapon/Weapon.kicad_pcb (KiCad board)
At the start: 2 copper layers, 97.3 x 61 mm, 34 parts, among them IC1 ATMEGA328-P, J1 MICRO_USB, P1 2P_CGRID_M, P2 USB-TTL, P3 2P_CGRID_M, Q1 NPN, Q2 NPN, U1 MCP73831, U2 RFID-RC522, U3 LM1084IT-3.3/NOPB, X1 16MHz

Commit message: Through Holes & Player/Health Schematic
I'm re-uploading the Apparel Sensor and Weapon PCBs with extended edges
and through holes on the corners for mounting. This also includes the
first draft of the Player/Health Schematic. Please critique
Other:
- board size 97.3 x 61 mm -> 97.3 x 68.5 mm
- board text added: "LaZIR Tag - April 2015"
- board text removed: "LaZIR Tag March 2015"
Changed lines of the file:
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@@
     (links 66)
     (no_connects 0)
-    (area 32.002999 22.92382 129.590001 85.1281)
+    (area 32.002999 20.079499 129.590001 88.632501)
     (thickness 1.6)
-    (drawings 13)
+    (drawings 21)
     (tracks 207)
     (zones 0)
@@
     )
   )
-  (gr_line (start 32.258 84.836) (end 129.54 84.836) (angle 90) (layer Edge.Cuts) (width 0.1))
-  (gr_line (start 129.54 23.876) (end 32.258 23.876) (angle 90) (layer Edge.Cuts) (width 0.1))
+  (gr_circle (center 127.3175 22.0345) (end 129.032 22.0345) (layer Edge.Cuts) (width 0.1))
+  (gr_circle (center 34.4805 22.0345) (end 36.195 22.0345) (layer Edge.Cuts) (width 0.1))
+  (gr_circle (center 34.4805 86.6775) (end 36.195 86.6775) (layer Edge.Cuts) (width 0.1))
+  (gr_circle (center 127.3175 86.6775) (end 129.032 86.6775) (layer Edge.Cuts) (width 0.1))
+  (gr_line (start 129.54 20.1295) (end 129.54 23.876) (angle 90) (layer Edge.Cuts) (width 0.1))
+  (gr_line (start 32.258 20.1295) (end 129.54 20.1295) (angle 90) (layer Edge.Cuts) (width 0.1))
+  (gr_line (start 32.258 23.876) (end 32.258 20.1295) (angle 90) (layer Edge.Cuts) (width 0.1))
+  (gr_line (start 129.54 88.5825) (end 129.54 84.836) (angle 90) (layer Edge.Cuts) (width 0.1))
+  (gr_line (start 32.258 88.5825) (end 129.54 88.5825) (angle 90) (layer Edge.Cuts) (width 0.1))
+  (gr_line (start 32.258 84.836) (end 32.258 88.5825) (angle 90) (layer Edge.Cuts) (width 0.1))
   (gr_line (start 129.54 23.876) (end 129.54 84.836) (angle 90) (layer Edge.Cuts) (width 0.1))
-  (gr_text "LaZIR Tag\nMarch 2015" (at 114.808 81.026) (layer B.SilkS)
+  (gr_text "LaZIR Tag - April 2015" (at 97.0915 86.614) (layer B.SilkS)
     (effects (font (size 1.5 1.5) (thickness 0.3)) (justify right mirror))
   )
-  (gr_text "Weapon PCB v1" (at 110.744 28.956) (layer B.SilkS)
+  (gr_text "Weapon PCB v1" (at 106.68 22.098) (layer B.SilkS)
     (effects (font (size 1.5 1.5) (thickness 0.3)) (justify right mirror))
   )
   (gr_line (start 32.258 84.836) (end 32.258 23.876) (angle 90) (layer Edge.Cuts) (width 0.1))
-  (gr_text "Weapon PCB v1" (at 128.524 28.956) (layer F.SilkS)
+  (gr_text "Weapon PCB v1" (at 124.3965 22.098) (layer F.SilkS)
     (effects (font (size 1.5 1.5) (thickness 0.3)) (justify right))
   )
-  (gr_text "LaZIR Tag\nMarch 2015" (at 128.27 81.026) (layer F.SilkS)
+  (gr_text "LaZIR Tag - April 2015" (at 124.2695 86.614) (layer F.SilkS)
     (effects (font (size 1.5 1.5) (thickness 0.3)) (justify right))
   )
@@
   (segment (start 92.329 57.658) (end 100.3808 49.6062) (width 0.508) (layer B.Cu) (net 1))
   (segment (start 88.773 24.384) (end 104.14 24.384) (width 0.508) (layer B.Cu) (net 2))
-  (segment (start 105.4608 25.92832) (end 105.4608 25.7048) (width 0.508) (layer B.Cu) (net 2) (status C00000))
-  (segment (start 105.4608 25.7048) (end 104.14 24.384) (width 0.508) (layer B.Cu) (net 2) (status 400000))
+  (segment (start 105.4608 25.92832) (end 105.4608 25.7048) (width 0.508) (layer B.Cu) (net 2))
+  (segment (start 105.4608 25.7048) (end 104.14 24.384) (width 0.508) (layer B.Cu) (net 2))
   (segment (start 34.417 74.2315) (end 37.338 74.2315) (width 0.254) (layer F.Cu) (net 2))
   (segment (start 38.9405 67.198) (end 37.807 67.198) (width 0.254) (layer F.Cu) (net 2))

Commit message: Quick Update #1 4/16
Parts:
- removed R7: 330, R4
Connections:
- LS1 pad 1: N-0000014 -> N-0000013
Routing:
- net N-0000013: track 3.94 -> 15.8 mm
- net N-0000014: track 10.3 -> 0.00 mm

Commit message: Quick Update #2 4/16
Parts:
- moved R10 0.09 mm to (87.5, 52.5), turned to 90 degrees
Routing:
- net +3.3V: track 51.6 -> 32.7 mm, vias 1 -> 0
- net Reset: track 16.7 -> 19.6 mm
Other:
- net class Default: trace_width 0.508 -> 0.254
Changed lines of the file:
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@@
     (thickness 1.6)
     (drawings 21)
-    (tracks 205)
+    (tracks 199)
     (zones 0)
     (modules 33)
@@
   )
   (setup
-    (last_trace_width 0.508)
+    (last_trace_width 0.254)
     (trace_clearance 0.254)
     (zone_clearance 0.508)
@@
   (net_class Default "This is the default net class."
     (clearance 0.254)
-    (trace_width 0.508)
+    (trace_width 0.254)
     (via_dia 0.889)
     (via_drill 0.635)
@@
     (descr "Transistor TO92 brochage type BC237")
     (tags "TR TO92")
-    (fp_text reference Q2 (at -1.27 3.81) (layer F.SilkS)
+    (fp_text reference Q2 (at -0.254 0.0254) (layer F.SilkS)
       (effects (font (size 1.016 1.016) (thickness 0.2032)))
     )
@@
   )
   (module R4 (layer F.Cu)
-    (at 87.4395 52.578 270)
+    (at 87.4776 52.5018 90)
     (descr "Resitance 4 pas")
     (tags R)
     (autoplace_cost180 10)
-    (fp_text reference R10 (at 0 0 270) (layer F.SilkS)
-      (effects (font (size 1.397 1.27) (thickness 0.2032)))
-    )
-    (fp_text value 10k (at 0 0 270) (layer F.SilkS) hide
+    (fp_text reference R10 (at 0 0 90) (layer F.SilkS)
+      (effects (font (size 1.397 1.27) (thickness 0.2032)))
+    )
+    (fp_text value 10k (at 0 0 90) (layer F.SilkS) hide
       (effects (font (size 1.397 1.27) (thickness 0.2032)))
     )
@@
     (fp_line (start -4.064 -0.508) (end -3.556 -1.016) (layer F.SilkS) (width 0.3048))
     (fp_line (start 5.08 0) (end 4.064 0) (layer F.SilkS) (width 0.3048))
-    (pad 1 thru_hole circle (at -5.08 0 270) (size 1.524 1.524) (drill 0.8128)
+    (pad 1 thru_hole circle (at -5.08 0 90) (size 1.524 1.524) (drill 0.8128)
       (layers *.Cu *.Mask F.SilkS)
       (net 21 Reset)
     )
-    (pad 2 thru_hole circle (at 5.08 0 270) (size 1.524 1.524) (drill 0.8128)
+    (pad 2 thru_hole circle (at 5.08 0 90) (size 1.524 1.524) (drill 0.8128)
       (layers *.Cu *.Mask F.SilkS)
       (net 1 +3.3V)
@@
   (gr_line (start 32.258 60.452) (end 70.358 60.452) (angle 90) (layer F.SilkS) (width 0.2))
   (gr_line (start 32.258 35.052) (end 32.258 60.452) (angle 90) (layer F.SilkS) (width 0.2))
-  (segment (start 100.3808 25.73782) (end 89.11082 25.73782) (width 0.508) (layer B.Cu) (net 1))
-  (segment (start 89.027 25.654) (end 89.027 25.7175) (width 0.254) (layer F.Cu) (net 1))
-  (via (at 89.027 25.654) (size 0.889) (layers F.Cu B.Cu) (net 1))
-  (segment (start 89.11082 25.73782) (end 89.027 25.654) (width 0.254) (layer B.Cu) (net 1))
-  (segment (start 87.4395 57.658) (end 92.329 57.658) (width 0.508) (layer B.Cu) (net 1))
-  (segment (start 100.3808 49.6062) (end 100.3808 25.73782) (width 0.508) (layer B.Cu) (net 1))
-  (segment (start 92.329 57.658) (end 100.3808 49.6062) (width 0.508) (layer B.Cu) (net 1))
+  (segment (start 87.4776 47.4218) (end 97.536 47.4218) (width 0.508) (layer B.Cu) (net 1) (status 400000))
+  (segment (start 100.3808 44.577) (end 100.3808 25.92832) (width 0.508) (layer B.Cu) (net 1) (status 800000))
+  (segment (start 97.536 47.4218) (end 100.3808 44.577) (width 0.508) (layer B.Cu) (net 1))
   (segment (start 88.773 24.384) (end 104.14 24.384) (width 0.508) (layer B.Cu) (net 2))
   (segment (start 105.4608 25.92832) (end 105.4608 25.7048) (width 0.508) (layer B.Cu) (net 2))
@@
   (segment (start 63.5635 80.137) (end 59.8805 80.137) (width 0.254) (layer B.Cu) (net 6))
   (segment (start 59.8805 80.137) (end 59.563 80.4545) (width 0.254) (layer B.Cu) (net 6))
-  (segment (start 57.023 80.4545) (end 57.023 71.5745) (width 0.508) (layer B.Cu) (net 7) (status 400000))
-  (segment (start 57.023 71.5745) (end 61.9125 66.685) (width 0.508) (layer B.Cu) (net 7) (status 800000))
+  (segment (start 57.023 80.4545) (end 57.023 71.5745) (width 0.508) (layer B.Cu) (net 7))
+  (segment (start 57.023 71.5745) (end 61.9125 66.685) (width 0.508) (layer B.Cu) (net 7))
   (segment (start 52.705 66.294) (end 52.705 64.262) (width 0.254) (layer B.Cu) (net 8))
   (segment (start 52.705 64.262) (end 54.864 62.103) (width 0.254) (layer B.Cu) (net 8))
@@
   (segment (start 88.392 71.374) (end 88.392 80.3275) (width 0.508) (layer F.Cu) (net 20))
   (via (at 88.392 71.374) (size 0.889) (layers F.Cu B.Cu) (net 20))
-  (segment (start 77.47 46.1645) (end 86.106 46.1645) (width 0.254) (layer B.Cu) (net 21))
-  (segment (start 87.4395 47.371) (end 87.4395 47.498) (width 0.254) (layer B.Cu) (net 21))
-  (segment (start 86.233 46.1645) (end 87.4395 47.371) (width 0.254) (layer B.Cu) (net 21))
-  (segment (start 86.106 46.1645) (end 86.233 46.1645) (width 0.254) (layer B.Cu) (net 21))
-  (segment (start 77.47 46.1645) (end 77.47 48.26) (width 0.254) (layer B.Cu) (net 21))
-  (segment (start 77.47 48.26) (end 77.216 48.514) (width 0.254) (layer B.Cu) (net 21))
+  (segment (start 87.4776 57.5818) (end 85.6996 57.5818) (width 0.254) (layer F.Cu) (net 21) (status 400000))
+  (segment (start 80.8482 52.1462) (end 77.216 48.514) (width 0.254) (layer F.Cu) (net 21) (status 800000))
+  (segment (start 80.8482 55.4482) (end 80.8482 52.1462) (width 0.254) (layer F.Cu) (net 21))
+  (segment (start 82.7532 57.3532) (end 80.8482 55.4482) (width 0.254) (layer F.Cu) (net 21))
+  (segment (start 85.471 57.3532) (end 82.7532 57.3532) (width 0.254) (layer F.Cu) (net 21))
+  (segment (start 85.6996 57.5818) (end 85.471 57.3532) (width 0.254) (layer F.Cu) (net 21))
   (segment (start 76.962 48.26) (end 77.216 48.514) (width 0.254) (layer B.Cu) (net 21))
   (segment (start 73.66 48.26) (end 76.962 48.26) (width 0.254) (layer B.Cu) (net 21))
@@
   (segment (start 45.0215 31.623) (end 40.132 31.623) (width 0.254) (layer B.Cu) (net 26))
   (segment (start 47.7012 64.3128) (end 47.7012 66.5099) (width 0.254) (layer F.Cu) (net 26))
-  (segment (start 85.852 61.214) (end 85.852 60.198) (width 0.254) (layer B.Cu) (net 27))
-  (segment (start 86.0425 35.052) (end 80.01 35.052) (width 0.254) (layer B.Cu) (net 27))
-  (segment (start 86.1695 34.925) (end 86.0425 35.052) (width 0.254) (layer B.Cu) (net 27))
-  (via (at 86.1695 34.925) (size 0.889) (layers F.Cu B.Cu) (net 27))
-  (segment (start 86.233 34.925) (end 86.1695 34.925) (width 0.254) (layer F.Cu) (net 27))
-  (segment (start 86.233 41.91) (end 86.233 34.925) (width 0.254) (layer F.Cu) (net 27))
-  (segment (start 86.487 44.196) (end 86.233 41.91) (width 0.254) (layer F.Cu) (net 27))
-  (segment (start 86.487 44.323) (end 86.487 44.196) (width 0.254) (layer F.Cu) (net 27))
-  (segment (start 86.0425 45.6565) (end 86.487 44.323) (width 0.254) (layer F.Cu) (net 27))
-  (segment (start 86.0425 51.2445) (end 86.0425 45.6565) (width 0.254) (layer F.Cu) (net 27))
-  (segment (start 85.979 51.181) (end 86.0425 51.2445) (width 0.254) (layer F.Cu) (net 27))
-  (segment (start 85.979 60.071) (end 85.979 51.181) (width 0.254) (layer F.Cu) (net 27))
-  (segment (start 85.852 60.198) (end 85.979 60.071) (width 0.254) (layer F.Cu) (net 27))
-  (via (at 85.852 60.198) (size 0.889) (layers F.Cu B.Cu) (net 27))
+  (segment (start 86.0806 61.214) (end 86.0806 49.7078) (width 0.254) (layer B.Cu) (net 27))
+  (segment (start 86.0298 35.052) (end 80.01 35.052) (width 0.254) (layer B.Cu) (net 27) (status 800000))
+  (segment (start 86.1568 34.925) (end 86.0298 35.052) (width 0.254) (layer B.Cu) (net 27))
+  (via (at 86.1568 34.925) (size 0.889) (layers F.Cu B.Cu) (net 27))
+  (segment (start 86.4616 35.2298) (end 86.1568 34.925) (width 0.254) (layer F.Cu) (net 27))
+  (segment (start 86.4616 45.0088) (end 86.4616 35.2298) (width 0.254) (layer F.Cu) (net 27))
+  (segment (start 86.0552 45.4152) (end 86.4616 45.0088) (width 0.254) (layer F.Cu) (net 27))
+  (segment (start 86.0552 49.53) (end 86.0552 45.4152) (width 0.254) (layer F.Cu) (net 27))
+  (segment (start 85.979 49.6062) (end 86.0552 49.53) (width 0.254) (layer F.Cu) (net 27))
+  (via (at 85.979 49.6062) (size 0.889) (layers F.Cu B.Cu) (net 27))
+  (segment (start 86.0806 49.7078) (end 85.979 49.6062) (width 0.254) (layer B.Cu) (net 27))
   (segment (start 84.836 61.214) (end 85.852 61.214) (width 0.254) (layer B.Cu) (net 27))
-  (segment (start 85.852 61.214) (end 86.2965 61.214) (width 0.254) (layer B.Cu) (net 27))
+  (segment (start 85.852 61.214) (end 86.0806 61.214) (width 0.254) (layer B.Cu) (net 27))
+  (segment (start 86.0806 61.214) (end 86.2965 61.214) (width 0.254) (layer B.Cu) (net 27))
   (segment (start 86.2965 61.214) (end 87.503 60.0075) (width 0.254) (layer B.Cu) (net 27))
   (zone (net 0) (net_name "") (layer F.Cu) (hatch edge 0.508)

Commit message: Quick Update #3 4/16
Parts:
- moved Q2 0.06 mm to (83.3, 39.6)
- moved R4 0.06 mm to (80.0, 29.9)
Routing:
- net Uart-Rx: track 25.2 -> 27.0 mm

Commit message: Quick Update #4 4/16
Routing:
- net V-Bat: track 192.9 -> 131.0 mm, vias 5 -> 4
Other:
- net class Default: trace_width 0.254 -> 0.508
Changed lines of the file:
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@@
     (thickness 1.6)
     (drawings 21)
-    (tracks 201)
+    (tracks 191)
     (zones 0)
     (modules 33)
@@
   )
   (setup
-    (last_trace_width 0.254)
+    (last_trace_width 0.508)
     (trace_clearance 0.254)
     (zone_clearance 0.508)
@@
   (net_class Default "This is the default net class."
     (clearance 0.254)
-    (trace_width 0.254)
+    (trace_width 0.508)
     (via_dia 0.889)
     (via_drill 0.635)
@@
   (segment (start 71.882 50.038) (end 71.882 52.578) (width 0.254) (layer F.Cu) (net 25))
   (via (at 71.882 50.038) (size 0.889) (layers F.Cu B.Cu) (net 25))
-  (segment (start 47.7266 64.1858) (end 47.7266 40.3606) (width 0.508) (layer B.Cu) (net 26))
-  (segment (start 47.7266 40.3606) (end 48.5902 39.497) (width 0.508) (layer B.Cu) (net 26))
-  (segment (start 47.7012 66.5099) (end 47.7012 64.2112) (width 0.508) (layer F.Cu) (net 26) (status 400000))
-  (segment (start 48.5902 39.497) (end 64.2366 39.497) (width 0.508) (layer B.Cu) (net 26))
-  (via (at 47.7266 64.1858) (size 0.889) (layers F.Cu B.Cu) (net 26))
-  (segment (start 47.7012 64.2112) (end 47.7266 64.1858) (width 0.508) (layer F.Cu) (net 26))
-  (segment (start 64.2366 39.497) (end 70.993 39.497) (width 0.508) (layer F.Cu) (net 26))
-  (via (at 64.2366 39.497) (size 0.889) (layers F.Cu B.Cu) (net 26))
-  (segment (start 70.993 39.497) (end 71.882 40.386) (width 0.508) (layer F.Cu) (net 26))
+  (segment (start 73.533 40.386) (end 68.6054 40.386) (width 0.508) (layer F.Cu) (net 26))
+  (segment (start 67.7164 39.497) (end 47.4218 39.497) (width 0.508) (layer B.Cu) (net 26))
+  (segment (start 68.6054 40.386) (end 67.7164 39.497) (width 0.508) (layer B.Cu) (net 26))
+  (via (at 68.6054 40.386) (size 0.889) (layers F.Cu B.Cu) (net 26))
+  (segment (start 51.181 74.295) (end 51.181 68.8086) (width 0.508) (layer F.Cu) (net 26))
+  (segment (start 48.8823 66.5099) (end 47.7012 66.5099) (width 0.508) (layer F.Cu) (net 26) (status 800000))
+  (segment (start 51.181 68.8086) (end 48.8823 66.5099) (width 0.508) (layer F.Cu) (net 26))
+  (segment (start 59.563 77.9145) (end 54.8005 77.9145) (width 0.508) (layer F.Cu) (net 26) (status 400000))
+  (segment (start 47.7012 66.5099) (end 47.3837 66.5099) (width 0.508) (layer F.Cu) (net 26) (status C00000))
+  (segment (start 47.3837 66.5099) (end 45.0596 64.1858) (width 0.508) (layer F.Cu) (net 26) (status 400000))
+  (via (at 45.0596 64.1858) (size 0.889) (layers F.Cu B.Cu) (net 26))
+  (segment (start 45.0596 64.1858) (end 45.0215 64.1477) (width 0.508) (layer B.Cu) (net 26))
+  (segment (start 45.0215 64.1477) (end 45.0215 37.0967) (width 0.508) (layer B.Cu) (net 26))
+  (via (at 73.533 40.386) (size 0.889) (layers F.Cu B.Cu) (net 26))
+  (segment (start 73.533 40.386) (end 73.533 43.307) (width 0.508) (layer B.Cu) (net 26))
+  (via (at 73.533 43.307) (size 0.889) (layers F.Cu B.Cu) (net 26))
+  (segment (start 73.533 43.307) (end 78.867 43.307) (width 0.508) (layer F.Cu) (net 26))
+  (segment (start 78.867 43.307) (end 79.502 43.942) (width 0.508) (layer F.Cu) (net 26))
   (segment (start 79.502 43.942) (end 80.264 43.942) (width 0.508) (layer F.Cu) (net 26))
-  (segment (start 78.867 43.307) (end 79.502 43.942) (width 0.508) (layer F.Cu) (net 26))
-  (segment (start 73.533 43.307) (end 78.867 43.307) (width 0.508) (layer F.Cu) (net 26))
-  (via (at 73.533 43.307) (size 0.889) (layers F.Cu B.Cu) (net 26))
-  (segment (start 73.533 40.386) (end 73.533 43.307) (width 0.508) (layer B.Cu) (net 26))
-  (via (at 73.533 40.386) (size 0.889) (layers F.Cu B.Cu) (net 26))
-  (segment (start 71.882 40.386) (end 73.533 40.386) (width 0.508) (layer F.Cu) (net 26))
+  (segment (start 47.4218 39.497) (end 45.0215 37.0967) (width 0.508) (layer B.Cu) (net 26))
+  (segment (start 82.0674 40.8432) (end 82.0674 40.0304) (width 0.508) (layer F.Cu) (net 26) (status 400000))
+  (segment (start 82.423 27.2288) (end 80.0354 24.8412) (width 0.508) (layer F.Cu) (net 26) (status 800000))
+  (segment (start 82.423 29.6672) (end 82.423 27.2288) (width 0.508) (layer F.Cu) (net 26))
+  (segment (start 83.3374 30.5816) (end 82.423 29.6672) (width 0.508) (layer F.Cu) (net 26))
+  (segment (start 83.3374 38.7604) (end 83.3374 30.5816) (width 0.508) (layer F.Cu) (net 26))
+  (segment (start 82.0674 40.0304) (end 83.3374 38.7604) (width 0.508) (layer F.Cu) (net 26))
   (segment (start 82.042 40.894) (end 82.042 42.164) (width 0.508) (layer B.Cu) (net 26))
   (segment (start 82.042 42.164) (end 80.264 43.942) (width 0.508) (layer B.Cu) (net 26))
-  (segment (start 46.6725 29.464) (end 49.403 29.464) (width 0.254) (layer B.Cu) (net 26))
+  (segment (start 46.6725 29.464) (end 49.403 29.464) (width 0.508) (layer B.Cu) (net 26))
   (segment (start 46.6725 29.464) (end 46.609 29.464) (width 0.254) (layer B.Cu) (net 26))
-  (segment (start 46.609 29.464) (end 46.609 31.496) (width 0.254) (layer B.Cu) (net 26))
+  (segment (start 46.609 29.464) (end 46.609 31.496) (width 0.508) (layer B.Cu) (net 26))
   (segment (start 46.609 31.496) (end 46.482 31.623) (width 0.254) (layer B.Cu) (net 26))
-  (segment (start 46.482 31.623) (end 45.0215 31.623) (width 0.254) (layer B.Cu) (net 26))
-  (segment (start 45.0215 31.623) (end 45.0215 64.262) (width 0.508) (layer B.Cu) (net 26))
-  (segment (start 47.3075 66.548) (end 47.6885 66.548) (width 0.254) (layer B.Cu) (net 26))
-  (segment (start 45.0215 64.262) (end 47.3075 66.548) (width 0.508) (layer B.Cu) (net 26))
-  (segment (start 47.7012 66.5099) (end 49.0474 66.5099) (width 0.254) (layer F.Cu) (net 26))
-  (segment (start 56.642 77.9145) (end 59.563 77.9145) (width 0.254) (layer F.Cu) (net 26))
-  (segment (start 54.8005 77.9145) (end 56.642 77.9145) (width 0.254) (layer F.Cu) (net 26))
-  (segment (start 51.181 74.295) (end 54.8005 77.9145) (width 0.254) (layer F.Cu) (net 26))
-  (segment (start 51.181 68.6435) (end 51.181 74.295) (width 0.254) (layer F.Cu) (net 26))
-  (segment (start 49.0474 66.5099) (end 51.181 68.6435) (width 0.254) (layer F.Cu) (net 26))
-  (segment (start 80.01 24.892) (end 82.2325 24.892) (width 0.254) (layer B.Cu) (net 26))
-  (segment (start 51.2445 29.464) (end 53.34 27.3685) (width 0.254) (layer B.Cu) (net 26))
-  (segment (start 53.34 27.3685) (end 53.34 24.4475) (width 0.254) (layer B.Cu) (net 26))
-  (segment (start 53.34 24.4475) (end 53.4035 24.384) (width 0.254) (layer B.Cu) (net 26))
-  (segment (start 53.4035 24.384) (end 79.502 24.384) (width 0.254) (layer B.Cu) (net 26))
-  (segment (start 79.502 24.384) (end 80.01 24.892) (width 0.254) (layer B.Cu) (net 26))
-  (segment (start 49.403 29.464) (end 51.2445 29.464) (width 0.254) (layer B.Cu) (net 26))
-  (segment (start 82.2325 24.892) (end 82.423 25.0825) (width 0.254) (layer B.Cu) (net 26))
-  (segment (start 82.423 25.0825) (end 82.423 32.893) (width 0.254) (layer B.Cu) (net 26))
-  (via (at 82.423 32.893) (size 0.889) (layers F.Cu B.Cu) (net 26))
-  (segment (start 82.423 32.893) (end 82.3595 32.9565) (width 0.254) (layer F.Cu) (net 26))
-  (segment (start 82.3595 32.9565) (end 82.3595 34.417) (width 0.508) (layer F.Cu) (net 26))
-  (segment (start 82.3595 34.417) (end 80.264 36.5125) (width 0.508) (layer F.Cu) (net 26))
-  (segment (start 80.264 36.5125) (end 80.264 43.942) (width 0.508) (layer F.Cu) (net 26))
-  (segment (start 40.132 31.623) (end 38.608 33.147) (width 0.254) (layer B.Cu) (net 26))
-  (segment (start 45.0215 31.623) (end 40.132 31.623) (width 0.254) (layer B.Cu) (net 26))
+  (segment (start 46.482 31.623) (end 45.0215 31.623) (width 0.508) (layer B.Cu) (net 26))
+  (segment (start 45.0215 31.623) (end 45.0215 37.0967) (width 0.508) (layer B.Cu) (net 26))
+  (segment (start 51.181 74.295) (end 54.8005 77.9145) (width 0.508) (layer F.Cu) (net 26))
+  (segment (start 40.132 31.623) (end 38.608 33.147) (width 0.508) (layer B.Cu) (net 26))
+  (segment (start 45.0215 31.623) (end 44.1706 31.623) (width 0.508) (layer B.Cu) (net 26))
+  (segment (start 44.1706 31.623) (end 40.132 31.623) (width 0.508) (layer B.Cu) (net 26))
   (segment (start 86.0806 61.214) (end 86.0806 49.7078) (width 0.254) (layer B.Cu) (net 27))
   (segment (start 86.0298 35.052) (end 80.01 35.052) (width 0.254) (layer B.Cu) (net 27))

Commit message: Quick Update #5 4/16
Routing:
- net GND: track 74.3 -> 55.6 mm, vias 2 -> 0
- net USBV: track 72.8 -> 76.6 mm
- net VoltageSense: track 36.0 -> 37.9 mm
- net V-Bat: track 131.0 -> 129.3 mm, vias 4 -> 2
Other:
- net class Default: via_drill 0.635 -> 0.508
