File: KiCad/Player-Health/Player-Health.sch (KiCad schematic (older format))
At the start: 21 parts, among them J1 MICRO_USB, U1 MCP73831

Commit message: Through Holes & Player/Health Schematic
I'm re-uploading the Apparel Sensor and Weapon PCBs with extended edges
and through holes on the corners for mounting. This also includes the
first draft of the Player/Health Schematic. Please critique
Parts:
- removed BT?: 400MAH_LIPO, symbol 400MAH_LIPO
- removed C? (x2): 10uF, ~, symbol C
- removed D?: RED, ~, symbol LED
- removed R? (x2): 220, ~, symbol R
- removed R?: 10k, ~, symbol R
- added C1, C7: 0.1uF, ~, symbol C
- added C3: 100uF, ~, symbol C
- added D1, D3, D4: LED, ~, symbol LED
- added M1: RUMBLE, symbol RUMBLE
- added P2: 6pM CGrid, symbol CONN_6
- added P3: 6pM Header, symbol CONN_6
- added P4: 6pF Header, symbol CONN_8
- added Q1: NPN, ~, symbol NPN
- added R2, R3, R8: 10k, ~, symbol R
- added R5: 560, ~, symbol R
- added R6: 1k, ~, symbol R
- added R7: 330, ~, symbol R
- added S1: SLIDESWITCH, ~, symbol SLIDESWITCH
- added U4: ESP8266, ~, symbol ESP8266
- gave numbers to parts that had none: 9
- renumbered C1 to C2, D1 to D2
Connections:
- net labels added: +3.3V, I2C CLK, I2C DAT, IR Sense, LED B, LED G, LED R, MISO, MOSI, Reset, Rumble, SCK, UART RX, UART TX, USBV, VBatt, VSense, WiFi Program
- wire segments 11 -> 82
Other:
- note added: "-3.3V Source\n-Voltage Sense\n-Status LEDs"
- note added: "-VBatt Source\n-USBV Source\n-Power Switch"
- note added: "3.3 V Regulator"
- note added: "AlphaNumeric Display"
- note added: "Connector to IR\nApparel Sensors"
- note added: "MicroController"
- note added: "Programming Port"
- note added: "RFID Reader"
- note added: "Rumble Motor"
- note added: "USB LiPo Charger"
- note added: "Wireless Device"
- moved on the sheet: C2, C4, C5, C6, D2, IC1, J1, P1, R1, R4, U1, U2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

Commit message: Quick Update #1 4/16
Parts:
- removed R7: 330, ~, symbol R
Connections:
- net UART RX: now also P3.4, U4.1 (TX); no longer U4.8 (RX)
- net UART TX: now also U4.8 (RX); no longer U4.1 (TX)
- net at Q1.1 (E): now also M1.1 (Vcc)
Changed lines of the file:
@@
 Sheet 1 1
 Title ""
-Date "10 apr 2015"
+Date "17 apr 2015"
 Rev ""
 Comp ""
@@
 Text GLabel 3250 6850 2    59   Output ~ 0
 UART TX
-Text GLabel 7800 6000 2    59   Output ~ 0
+Text GLabel 7800 6700 2    59   Output ~ 0
 UART RX
 Text Notes 2000 4800 2    118  ~ 0
@@
 	1    0    0    -1
 $EndComp
-Text GLabel 7800 6700 2    59   Input ~ 0
+Text GLabel 7800 6000 2    59   Input ~ 0
 UART TX
 $Comp
@@
 $EndComp
 $Comp
-L R R7
-U 1 1 552837A1
-P 7400 2000
-F 0 "R7" V 7480 2000 40  0000 C CNN
-F 1 "330" V 7407 2001 40  0000 C CNN
-F 2 "~" V 7330 2000 30  0000 C CNN
-F 3 "~" H 7400 2000 30  0000 C CNN
-	1    7400 2000
-	0    -1   -1   0
-$EndComp
-$Comp
 L LED D4
 U 1 1 552837A7
@@
 	6500 1200 6500 1250
 Wire Wire Line
-	7150 2000 7000 2000
+	7000 2000 7650 2000
 Text Notes 6900 750  2    118  ~ 0
 Rumble Motor
@@
 	1    0    0    -1
 $EndComp
+Wire Wire Line
+	10250 4000 9800 4000
 $EndSCHEMATC

Commit message: Quick Update #1 4/17
Finished PCBs for Apparel Sensor and Weapon, ready for review
Finished Schematic, Netlist, and Component Assignment for Player/Health
Started PCB with components and text for Player/Health
New Component footprints for 8x1 pin array, wifi module, and
alphanumeric
Parts:
- P4: value 6pF Header -> 8pF Header
- renumbered R8 to R7
Changed lines of the file:
@@
 $EndComp
 $Comp
-L GND #PWR4
+L GND #PWR01
 U 1 1 5501101E
 P 1850 2050
-F 0 "#PWR4" H 1850 2050 30  0001 C CNN
+F 0 "#PWR01" H 1850 2050 30  0001 C CNN
 F 1 "GND" H 1850 1980 30  0001 C CNN
 F 2 "" H 1850 2050 60  0000 C CNN
@@
 $EndComp
 $Comp
-L GND #PWR9
+L GND #PWR02
 U 1 1 55011447
 P 3950 2300
-F 0 "#PWR9" H 3950 2300 30  0001 C CNN
+F 0 "#PWR02" H 3950 2300 30  0001 C CNN
 F 1 "GND" H 3950 2230 30  0001 C CNN
 F 2 "" H 3950 2300 60  0000 C CNN
@@
 $EndComp
 $Comp
-L GND #PWR7
+L GND #PWR03
 U 1 1 550112D9
 P 3700 2300
-F 0 "#PWR7" H 3700 2300 30  0001 C CNN
+F 0 "#PWR03" H 3700 2300 30  0001 C CNN
 F 1 "GND" H 3700 2230 30  0001 C CNN
 F 2 "" H 3700 2300 60  0000 C CNN
@@
 $EndComp
 $Comp
-L GND #PWR6
+L GND #PWR04
 U 1 1 5501126E
 P 3550 1800
-F 0 "#PWR6" H 3550 1800 30  0001 C CNN
+F 0 "#PWR04" H 3550 1800 30  0001 C CNN
 F 1 "GND" H 3550 1730 30  0001 C CNN
 F 2 "" H 3550 1800 60  0000 C CNN
@@
 $EndComp
 $Comp
-L GND #PWR3
+L GND #PWR05
 U 1 1 55011060
 P 1650 1800
-F 0 "#PWR3" H 1650 1800 30  0001 C CNN
+F 0 "#PWR05" H 1650 1800 30  0001 C CNN
 F 1 "GND" H 1650 1730 30  0001 C CNN
 F 2 "" H 1650 1800 60  0000 C CNN
@@
 $EndComp
 $Comp
-L GND #PWR8
+L GND #PWR06
 U 1 1 55280CC3
 P 3800 1150
-F 0 "#PWR8" H 3800 1150 30  0001 C CNN
+F 0 "#PWR06" H 3800 1150 30  0001 C CNN
 F 1 "GND" H 3800 1080 30  0001 C CNN
 F 2 "" H 3800 1150 60  0000 C CNN
@@
 VSense
 $Comp
-L +3.3V #PWR10
+L +3.3V #PWR07
 U 1 1 55280D8C
 P 4050 3800
-F 0 "#PWR10" H 4050 3760 30  0001 C CNN
+F 0 "#PWR07" H 4050 3760 30  0001 C CNN
 F 1 "+3.3V" H 4050 3910 30  0000 C CNN
 F 2 "" H 4050 3800 60  0000 C CNN
@@
 $EndComp
 $Comp
-L GND #PWR5
+L GND #PWR08
 U 1 1 55280D9B
 P 3300 4150
-F 0 "#PWR5" H 3300 4150 30  0001 C CNN
+F 0 "#PWR08" H 3300 4150 30  0001 C CNN
 F 1 "GND" H 3300 4080 30  0001 C CNN
 F 2 "" H 3300 4150 60  0000 C CNN
@@
 VBatt
 $Comp
-L GND #PWR12
+L GND #PWR09
 U 1 1 55281188
 P 7650 3850
-F 0 "#PWR12" H 7650 3850 30  0001 C CNN
+F 0 "#PWR09" H 7650 3850 30  0001 C CNN
 F 1 "GND" H 7650 3780 30  0001 C CNN
 F 2 "" H 7650 3850 60  0000 C CNN
@@
 I2C DAT
 $Comp
-L +3.3V #PWR1
+L +3.3V #PWR010
 U 1 1 552816BB
 P 1250 5150
-F 0 "#PWR1" H 1250 5110 30  0001 C CNN
+F 0 "#PWR010" H 1250 5110 30  0001 C CNN
 F 1 "+3.3V" H 1250 5260 30  0000 C CNN
 F 2 "" H 1250 5150 60  0000 C CNN
@@
 $EndComp
 $Comp
-L GND #PWR2
+L GND #PWR011
 U 1 1 55281865
 P 1250 7500
-F 0 "#PWR2" H 1250 7500 30  0001 C CNN
+F 0 "#PWR011" H 1250 7500 30  0001 C CNN
 F 1 "GND" H 1250 7430 30  0001 C CNN
 F 2 "" H 1250 7500 60  0000 C CNN
@@
 Reset
 $Comp
-L GND #PWR11
+L GND #PWR012
 U 1 1 55281D1D
 P 4500 6500
-F 0 "#PWR11" H 4500 6500 30  0001 C CNN
+F 0 "#PWR012" H 4500 6500 30  0001 C CNN
 F 1 "GND" H 4500 6430 30  0001 C CNN
 F 2 "" H 4500 6500 60  0000 C CNN
@@
 UART TX
 $Comp
-L GND #PWR16
+L GND #PWR013
 U 1 1 552825A2
 P 7950 6500
-F 0 "#PWR16" H 7950 6500 30  0001 C CNN
+F 0 "#PWR013" H 7950 6500 30  0001 C CNN
 F 1 "GND" H 7950 6430 30  0001 C CNN
 F 2 "" H 7950 6500 60  0000 C CNN
@@
 $EndComp
 $Comp
-L +3.3V #PWR14
+L +3.3V #PWR014
 U 1 1 552825B1
 P 7650 6500
-F 0 "#PWR14" H 7650 6460 30  0001 C CNN
+F 0 "#PWR014" H 7650 6460 30  0001 C CNN
 F 1 "+3.3V" H 7650 6610 30  0000 C CNN
 F 2 "" H 7650 6500 60  0000 C CNN
@@
 $EndComp
 $Comp
-L +3.3V #PWR13
+L +3.3V #PWR015
 U 1 1 55282851
 P 7650 6100
-F 0 "#PWR13" H 7650 6060 30  0001 C CNN
+F 0 "#PWR015" H 7650 6060 30  0001 C CNN
 F 1 "+3.3V" H 7650 6210 30  0000 C CNN
 F 2 "" H 7650 6100 60  0000 C CNN
@@
 $EndComp
 $Comp
-L GND #PWR19
+L GND #PWR016
 U 1 1 55282A83
 P 9750 1850
-F 0 "#PWR19" H 9750 1850 30  0001 C CNN
+F 0 "#PWR016" H 9750 1850 30  0001 C CNN
 F 1 "GND" H 9750 1780 30  0001 C CNN
 F 2 "" H 9750 1850 60  0000 C CNN
@@
 $EndComp
 $Comp
-L +3.3V #PWR18
+L +3.3V #PWR017
 U 1 1 55282A89
 P 9750 1750
-F 0 "#PWR18" H 9750 1710 30  0001 C CNN
+F 0 "#PWR017" H 9750 1710 30  0001 C CNN
 F 1 "+3.3V" H 9750 1860 30  0000 C CNN
 F 2 "" H 9750 1750 60  0000 C CNN
@@
 MOSI
 $Comp
-L GND #PWR22
+L GND #PWR018
 U 1 1 55282C20
 P 10200 6100
-F 0 "#PWR22" H 10200 6100 30  0001 C CNN
+F 0 "#PWR018" H 10200 6100 30  0001 C CNN
 F 1 "GND" H 10200 6030 30  0001 C CNN
 F 2 "" H 10200 6100 60  0000 C CNN
@@
 $EndComp
 $Comp
-L +3.3V #PWR21
+L +3.3V #PWR019
 U 1 1 55282C26
 P 10200 5900
-F 0 "#PWR21" H 10200 5860 30  0001 C CNN
+F 0 "#PWR019" H 10200 5860 30  0001 C CNN
 F 1 "+3.3V" H 10200 6010 30  0000 C CNN
 F 2 "" H 10200 5900 60  0000 C CNN
@@
 P 9550 6250
 F 0 "P4" V 9500 6250 60  0000 C CNN
-F 1 "6pF Header" V 9600 6250 60  0000 C CNN
+F 1 "8pF Header" V 9600 6250 60  0000 C CNN
 F 2 "" H 9550 6250 60  0000 C CNN
 F 3 "" H 9550 6250 60  0000 C CNN
@@
 $EndComp
 $Comp
-L GND #PWR20
+L GND #PWR020
 U 1 1 55282D84
 P 10100 4300
-F 0 "#PWR20" H 10100 4300 30  0001 C CNN
+F 0 "#PWR020" H 10100 4300 30  0001 C CNN
 F 1 "GND" H 10100 4230 30  0001 C CNN
 F 2 "" H 10100 4300 60  0000 C CNN
@@
 $EndComp
 $Comp
-L R R8
+L R R7
 U 1 1 55282E5A
 P 10250 3400
-F 0 "R8" V 10330 3400 40  0000 C CNN
+F 0 "R7" V 10330 3400 40  0000 C CNN
 F 1 "10k" V 10257 3401 40  0000 C CNN
 F 2 "~" V 10180 3400 30  0000 C CNN
@@
 $EndComp
 $Comp
-L +3.3V #PWR23
+L +3.3V #PWR021
 U 1 1 55282FA8
 P 10600 3400
-F 0 "#PWR23" H 10600 3360 30  0001 C CNN
+F 0 "#PWR021" H 10600 3360 30  0001 C CNN
 F 1 "+3.3V" H 10600 3510 30  0000 C CNN
 F 2 "" H 10600 3400 60  0000 C CNN
@@
 Rumble
 $Comp
-L GND #PWR17
+L GND #PWR022
 U 1 1 55283776
 P 8050 2000
-F 0 "#PWR17" H 8050 2000 30  0001 C CNN
+F 0 "#PWR022" H 8050 2000 30  0001 C CNN
 F 1 "GND" H 8050 1930 30  0001 C CNN
 F 2 "" H 8050 2000 60  0000 C CNN
@@
 $EndComp
 $Comp
-L GND #PWR15
+L GND #PWR023
 U 1 1 552837AD
 P 7800 1200
-F 0 "#PWR15" H 7800 1200 30  0001 C CNN
+F 0 "#PWR023" H 7800 1200 30  0001 C CNN
 F 1 "GND" H 7800 1130 30  0001 C CNN
 F 2 "" H 7800 1200 60  0000 C CNN

Commit message: Quick Update #2 4/17
Added Jumpers to Schematic, Net List and PCB, but failing connectivity
Parts:
- added JP1, JP2: JUMPER, symbol JUMPER
Connections:
- net GND: now also JP2.2
- net UART RX: now also JP1.2
- net UART TX: now also JP1.1
- net WiFi Program: no longer names the net of U4.6 (GPIO_0)
- net WiFi Program: now also JP2.1
Changed lines of the file:
@@
 Text GLabel 3500 5550 2    59   Input ~ 0
 MISO
-Text GLabel 3250 6850 2    59   Output ~ 0
+Text GLabel 3950 7100 2    59   Output ~ 0
 UART TX
 Text GLabel 7800 6700 2    59   Output ~ 0
@@
 	0    1    1    0
 $EndComp
-Text GLabel 7800 6200 2    59   Input ~ 0
-WiFi Program
 Text Notes 5700 5300 0    118  ~ 0
 Wireless Device
@@
 Text GLabel 3200 6000 2    60   Input ~ 0
 VSense
-Text GLabel 3650 6750 2    59   Input ~ 0
+Text GLabel 3950 6650 2    59   Input ~ 0
 UART RX
 $Comp
@@
 	3250 5650 3200 5650
 Wire Wire Line
-	3250 6850 3200 6850
+	3200 6850 3650 6850
 Wire Wire Line
 	3200 5750 4800 5750
@@
 Wire Wire Line
 	10250 4000 9800 4000
+$Comp
+L GND #PWR024
+U 1 1 5530A16F
+P 8300 6200
+F 0 "#PWR024" H 8300 6200 30  0001 C CNN
+F 1 "GND" H 8300 6130 30  0001 C CNN
+F 2 "" H 8300 6200 60  0000 C CNN
+F 3 "" H 8300 6200 60  0000 C CNN
+	1    8300 6200
+	0    -1   -1   0
+$EndComp
+$Comp
+L JUMPER JP2
+U 1 1 5530A41F
+P 8050 6200
+F 0 "JP2" H 8050 6100 60  0000 C CNN
+F 1 "JUMPER" H 8050 6300 60  0000 C CNN
+F 2 "" H 8050 6200 60  0000 C CNN
+F 3 "" H 8050 6200 60  0000 C CNN
+	1    8050 6200
+	1    0    0    -1
+$EndComp
+Wire Wire Line
+	8250 6200 8300 6200
+$Comp
+L JUMPER JP1
+U 1 1 5530A4A4
+P 3850 6850
+F 0 "JP1" H 3850 6750 60  0000 C CNN
+F 1 "JUMPER" H 3850 6950 60  0000 C CNN
+F 2 "" H 3850 6850 60  0000 C CNN
+F 3 "" H 3850 6850 60  0000 C CNN
+	1    3850 6850
+	0    -1   -1   0
+$EndComp
+Wire Wire Line
+	3650 7100 3950 7100
+Wire Wire Line
+	3650 6650 3950 6650
+Wire Wire Line
+	3650 6650 3650 6750
+Connection ~ 3850 6650
+Wire Wire Line
+	3650 6850 3650 7100
+Connection ~ 3850 7100
 $EndSCHEMATC

Commit message: Quick Update #3 4/17
Connections:
- net UART RX: no longer JP1.2
- net UART TX: no longer IC1.3 ((PCINT17/TXD)PD1)
- new net: IC1.3 ((PCINT17/TXD)PD1), JP1.2
Other:
- moved on the sheet: JP1
Changed lines of the file:
@@
 Text GLabel 3500 5550 2    59   Input ~ 0
 MISO
-Text GLabel 3950 7100 2    59   Output ~ 0
+Text GLabel 3800 6950 2    59   Output ~ 0
 UART TX
 Text GLabel 7800 6700 2    59   Output ~ 0
@@
 Text GLabel 3200 6000 2    60   Input ~ 0
 VSense
-Text GLabel 3950 6650 2    59   Input ~ 0
+Text GLabel 3250 6750 2    59   Input ~ 0
 UART RX
 $Comp
@@
 	0    -1   -1   0
 $EndComp
-Connection ~ 2150 1550
-Wire Wire Line
-	1550 1700 1650 1700
-Wire Wire Line
-	1650 1700 1650 1800
-Wire Wire Line
-	1850 1950 1850 2050
-Connection ~ 1850 1550
-Wire Wire Line
-	2000 1550 2000 1350
-Connection ~ 2000 1550
-Wire Wire Line
-	1550 1550 2350 1550
-Wire Wire Line
-	2150 2050 2350 2050
-Wire Wire Line
-	3550 1700 3550 1800
-Wire Wire Line
-	3550 1600 3700 1600
-Wire Wire Line
-	3700 1600 3700 1700
-Wire Wire Line
-	3700 2200 3700 2300
-Wire Wire Line
-	3950 2200 3950 2300
-Wire Wire Line
-	3700 1150 3800 1150
-Wire Wire Line
-	3950 1250 3950 1800
-Wire Wire Line
-	3950 1500 3550 1500
-Wire Wire Line
-	3700 950  3950 950
-Connection ~ 3950 1500
-Wire Wire Line
-	3950 1350 3750 1350
-Connection ~ 3950 1350
-Wire Notes Line
-	500  2700 5600 2700
-Wire Notes Line
-	5600 500  5600 7800
-Wire Wire Line
-	2500 3300 2900 3300
-Wire Wire Line
-	2750 3400 2750 3300
-Connection ~ 2750 3300
-Wire Wire Line
-	2750 3900 2750 4000
-Connection ~ 2750 4000
-Wire Wire Line
-	3300 3600 3300 4150
-Connection ~ 3300 4000
-Wire Wire Line
-	2800 4000 2600 4000
-Wire Wire Line
-	3700 3500 3700 3300
-Wire Wire Line
-	3700 3300 4050 3300
-Wire Wire Line
-	3700 3900 3700 4000
-Wire Wire Line
-	3700 4000 3300 4000
-Wire Wire Line
-	7650 3550 7400 3550
-Wire Wire Line
-	7550 3550 7550 3700
-Wire Wire Line
-	7550 3700 7400 3700
-Connection ~ 7550 3550
-Wire Wire Line
-	7400 3850 7650 3850
-Wire Wire Line
-	7650 4150 7400 4150
-Wire Wire Line
-	7400 4000 7650 4000
-Wire Wire Line
-	2000 3300 2100 3300
-Wire Wire Line
-	4050 3700 4050 3800
-Wire Notes Line
-	500  4550 5600 4550
-Wire Wire Line
-	3250 6400 3200 6400
-Wire Wire Line
-	1250 6050 1250 5150
-Connection ~ 1250 5150
-Wire Wire Line
-	1250 6450 1250 7500
-Connection ~ 1250 7350
-Connection ~ 1250 7450
-Wire Wire Line
-	1250 5150 1300 5150
-Wire Wire Line
-	1300 7350 1250 7350
-Wire Wire Line
-	1300 7450 1250 7450
-Wire Wire Line
-	3250 6600 3200 6600
-Wire Wire Line
-	3200 7350 3250 7350
-Wire Wire Line
-	3250 5250 3200 5250
-Wire Wire Line
-	3600 5350 3200 5350
-Wire Wire Line
-	3650 6500 3200 6500
-Wire Wire Line
-	4200 6450 4800 6450
-Wire Wire Line
-	4500 6450 4500 6500
-Connection ~ 4500 6450
-Wire Wire Line
-	3250 5450 3200 5450
-Wire Wire Line
-	3250 5650 3200 5650
-Wire Wire Line
-	3200 6850 3650 6850
-Wire Wire Line
-	3200 5750 4800 5750
-Wire Wire Line
-	4800 5750 4800 6050
-Wire Wire Line
-	3200 5850 4200 5850
-Wire Wire Line
-	4200 5850 4200 6050
-Wire Wire Line
-	3200 7250 3600 7250
-Wire Wire Line
-	3650 6750 3200 6750
-Wire Wire Line
-	3500 5550 3200 5550
-Wire Wire Line
-	3550 5150 3200 5150
-Wire Wire Line
-	7800 6700 7650 6700
-Wire Wire Line
-	7650 6000 7800 6000
-Wire Wire Line
-	7950 6500 7950 6600
-Wire Wire Line
-	7950 6600 7650 6600
-Wire Wire Line
-	7800 6200 7650 6200
-Wire Wire Line
-	9750 1650 10100 1650
-Wire Wire Line
-	10100 1450 9750 1450
-Wire Wire Line
-	10200 6400 9900 6400
-Wire Wire Line
-	10200 6100 9900 6100
-Wire Wire Line
-	9900 5900 10200 5900
-Wire Wire Line
-	10100 4300 9800 4300
-Wire Wire Line
-	9800 4200 9950 4200
-Wire Wire Line
-	9950 4200 9950 4300
-Connection ~ 9950 4300
-Wire Wire Line
-	9900 3800 9800 3800
-Connection ~ 9900 3400
-Wire Wire Line
-	9600 3400 10000 3400
-Wire Wire Line
-	10500 3400 10600 3400
-Wire Notes Line
-	5600 5050 11200 5050
-Wire Notes Line
-	5600 2550 11200 2550
-Wire Notes Line
-	8700 500  8700 7200
-Wire Wire Line
-	6350 1200 6600 1200
-Connection ~ 6500 1200
-Wire Wire Line
-	7100 1200 7250 1200
-Wire Wire Line
-	7650 1200 7800 1200
-Wire Wire Line
-	7150 1450 7000 1450
-Wire Wire Line
-	7000 1450 7000 1600
-Wire Wire Line
-	6700 1800 6500 1800
-Wire Wire Line
-	6500 1800 6500 1750
-Wire Wire Line
-	6500 1200 6500 1250
-Wire Wire Line
-	7000 2000 7650 2000
 Text Notes 6900 750  2    118  ~ 0
 Rumble Motor
@@
 	1    0    0    -1
 $EndComp
-Wire Wire Line
-	10250 4000 9800 4000
 $Comp
 L GND #PWR024
 U 1 1 5530A16F
-P 8300 6200
-F 0 "#PWR024" H 8300 6200 30  0001 C CNN
-F 1 "GND" H 8300 6130 30  0001 C CNN
-F 2 "" H 8300 6200 60  0000 C CNN
-F 3 "" H 8300 6200 60  0000 C CNN
-	1    8300 6200
+P 8350 6200
+F 0 "#PWR024" H 8350 6200 30  0001 C CNN
+F 1 "GND" H 8350 6130 30  0001 C CNN
+F 2 "" H 8350 6200 60  0000 C CNN
+F 3 "" H 8350 6200 60  0000 C CNN
+	1    8350 6200
 	0    -1   -1   0
 $EndComp
@@
 	1    0    0    -1
 $EndComp
-Wire Wire Line
-	8250 6200 8300 6200
 $Comp
 L JUMPER JP1
 U 1 1 5530A4A4
-P 3850 6850
-F 0 "JP1" H 3850 6750 60  0000 C CNN
-F 1 "JUMPER" H 3850 6950 60  0000 C CNN
-F 2 "" H 3850 6850 60  0000 C CNN
-F 3 "" H 3850 6850 60  0000 C CNN
-	1    3850 6850
-	0    -1   -1   0
-$EndComp
-Wire Wire Line
-	3650 7100 3950 7100
-Wire Wire Line
-	3650 6650 3950 6650
-Wire Wire Line
-	3650 6650 3650 6750
-Connection ~ 3850 6650
-Wire Wire Line
-	3650 6850 3650 7100
-Connection ~ 3850 7100
+P 3500 6950
+F 0 "JP1" H 3500 6850 60  0000 C CNN
+F 1 "JUMPER" H 3500 7050 60  0000 C CNN
+F 2 "" H 3500 6950 60  0000 C CNN
+F 3 "" H 3500 6950 60  0000 C CNN
+	1    3500 6950
+	-1   0    0    1
+$EndComp
+Connection ~ 2150 1550
+Wire Wire Line
+	1550 1700 1650 1700
+Wire Wire Line
+	1650 1700 1650 1800
+Wire Wire Line
+	1850 1950 1850 2050
+Connection ~ 1850 1550
+Wire Wire Line
+	2000 1550 2000 1350
+Connection ~ 2000 1550
+Wire Wire Line
+	1550 1550 2350 1550
+Wire Wire Line
+	2150 2050 2350 2050
+Wire Wire Line
+	3550 1700 3550 1800
+Wire Wire Line
+	3550 1600 3700 1600
+Wire Wire Line
+	3700 1600 3700 1700
+Wire Wire Line
+	3700 2200 3700 2300
+Wire Wire Line
+	3950 2200 3950 2300
+Wire Wire Line
+	3700 1150 3800 1150
+Wire Wire Line
+	3950 1250 3950 1800
+Wire Wire Line
+	3950 1500 3550 1500
+Wire Wire Line
+	3700 950  3950 950
+Connection ~ 3950 1500
+Wire Wire Line
+	3950 1350 3750 1350
+Connection ~ 3950 1350
+Wire Notes Line
+	500  2700 5600 2700
+Wire Notes Line
+	5600 500  5600 7800
+Wire Wire Line
+	2500 3300 2900 3300
+Wire Wire Line
+	2750 3400 2750 3300
+Connection ~ 2750 3300
+Wire Wire Line
+	2750 3900 2750 4000
+Connection ~ 2750 4000
+Wire Wire Line
+	3300 3600 3300 4150
+Connection ~ 3300 4000
+Wire Wire Line
+	2800 4000 2600 4000
+Wire Wire Line
+	3700 3500 3700 3300
+Wire Wire Line
+	3700 3300 4050 3300
+Wire Wire Line
+	3700 3900 3700 4000
+Wire Wire Line
+	3700 4000 3300 4000
+Wire Wire Line
+	7650 3550 7400 3550
+Wire Wire Line
+	7550 3550 7550 3700
+Wire Wire Line
+	7550 3700 7400 3700
+Connection ~ 7550 3550
+Wire Wire Line
+	7400 3850 7650 3850
+Wire Wire Line
+	7650 4150 7400 4150
+Wire Wire Line
+	7400 4000 7650 4000
+Wire Wire Line
+	2000 3300 2100 3300
+Wire Wire Line
+	4050 3700 4050 3800
+Wire Notes Line
+	500  4550 5600 4550
+Wire Wire Line
+	3250 6400 3200 6400
+Wire Wire Line
+	1250 6050 1250 5150
+Connection ~ 1250 5150
+Wire Wire Line
+	1250 6450 1250 7500
+Connection ~ 1250 7350
+Connection ~ 1250 7450
+Wire Wire Line
+	1250 5150 1300 5150
+Wire Wire Line
+	1300 7350 1250 7350
+Wire Wire Line
+	1300 7450 1250 7450
+Wire Wire Line
+	3250 6600 3200 6600
+Wire Wire Line
+	3200 7350 3250 7350
+Wire Wire Line
+	3250 5250 3200 5250
+Wire Wire Line
+	3600 5350 3200 5350
+Wire Wire Line
+	3650 6500 3200 6500
+Wire Wire Line
+	4200 6450 4800 6450
+Wire Wire Line
+	4500 6450 4500 6500
+Connection ~ 4500 6450
+Wire Wire Line
+	3250 5450 3200 5450
+Wire Wire Line
+	3250 5650 3200 5650
+Wire Wire Line
+	3200 5750 4800 5750
+Wire Wire Line
+	4800 5750 4800 6050
+Wire Wire Line
+	3200 5850 4200 5850
+Wire Wire Line
+	4200 5850 4200 6050
+Wire Wire Line
+	3200 7250 3600 7250
+Wire Wire Line
+	3500 5550 3200 5550
+Wire Wire Line
+	3550 5150 3200 5150
+Wire Wire Line
+	7800 6700 7650 6700
+Wire Wire Line
+	7650 6000 7800 6000
+Wire Wire Line
+	7950 6500 7950 6600
+Wire Wire Line
+	7950 6600 7650 6600
+Wire Wire Line
+	7800 6200 7650 6200
+Wire Wire Line
+	9750 1650 10100 1650
+Wire Wire Line
+	10100 1450 9750 1450
+Wire Wire Line
+	10200 6400 9900 6400
+Wire Wire Line
+	10200 6100 9900 6100
+Wire Wire Line
+	9900 5900 10200 5900
+Wire Wire Line
+	10100 4300 9800 4300
+Wire Wire Line
+	9800 4200 9950 4200
+Wire Wire Line
+	9950 4200 9950 4300
+Connection ~ 9950 4300
+Wire Wire Line
+	9900 3800 9800 3800
+Connection ~ 9900 3400
+Wire Wire Line
+	9600 3400 10000 3400
+Wire Wire Line
+	10500 3400 10600 3400
+Wire Notes Line
+	5600 5050 11200 5050
+Wire Notes Line
+	5600 2550 11200 2550
+Wire Notes Line
+	8700 500  8700 7200
+Wire Wire Line
+	6350 1200 6600 1200
+Connection ~ 6500 1200
+Wire Wire Line
+	7100 1200 7250 1200
+Wire Wire Line
+	7650 1200 7800 1200
+Wire Wire Line
+	7150 1450 7000 1450
+Wire Wire Line
+	7000 1450 7000 1600
+Wire Wire Line
+	6700 1800 6500 1800
+Wire Wire Line
+	6500 1800 6500 1750
+Wire Wire Line
+	6500 1200 6500 1250
+Wire Wire Line
+	7000 2000 7650 2000
+Wire Wire Line
+	10250 4000 9800 4000
+Wire Wire Line
+	8250 6200 8350 6200
+Wire Wire Line
+	3250 6750 3200 6750
+Wire Wire Line
+	3300 6950 3250 6950
+Wire Wire Line
+	3250 6950 3250 6850
+Wire Wire Line
+	3250 6850 3200 6850
+Wire Wire Line
+	3800 6950 3750 6950
 $EndSCHEMATC
