File: KiCad/Player-Health/Player-Health.sch (KiCad schematic (older format))
At the start: 34 parts, among them IC1 ATMEGA328-P, J1 MICRO_USB, M1 RUMBLE, P1 2P_CGRID_M, P2 6pM CGrid, P3 6pM Header, P4 8pF Header, Q1 NPN, U1 MCP73831, U2 LM1084IT-3.3/NOPB, U3 14SLED, U4 ESP8266, X1 CRYSTAL

Commit message: Last Update for the Night 4/17(4/16)
General PCB layout, fix to jumper pads
Parts:
- JP1: footprint (none) -> ~
Connections:
- net UART TX: now also JP1.2; no longer JP1.1
- net at IC1.3 ((PCINT17/TXD)PD1): now also JP1.1; no longer JP1.2
Changed lines of the file:
@@
 $EndComp
 $Comp
-L GND #PWR01
+L GND #PWR4
 U 1 1 5501101E
 P 1850 2050
-F 0 "#PWR01" H 1850 2050 30  0001 C CNN
+F 0 "#PWR4" H 1850 2050 30  0001 C CNN
 F 1 "GND" H 1850 1980 30  0001 C CNN
 F 2 "" H 1850 2050 60  0000 C CNN
@@
 $EndComp
 $Comp
-L GND #PWR02
+L GND #PWR9
 U 1 1 55011447
 P 3950 2300
-F 0 "#PWR02" H 3950 2300 30  0001 C CNN
+F 0 "#PWR9" H 3950 2300 30  0001 C CNN
 F 1 "GND" H 3950 2230 30  0001 C CNN
 F 2 "" H 3950 2300 60  0000 C CNN
@@
 $EndComp
 $Comp
-L GND #PWR03
+L GND #PWR7
 U 1 1 550112D9
 P 3700 2300
-F 0 "#PWR03" H 3700 2300 30  0001 C CNN
+F 0 "#PWR7" H 3700 2300 30  0001 C CNN
 F 1 "GND" H 3700 2230 30  0001 C CNN
 F 2 "" H 3700 2300 60  0000 C CNN
@@
 $EndComp
 $Comp
-L GND #PWR04
+L GND #PWR6
 U 1 1 5501126E
 P 3550 1800
-F 0 "#PWR04" H 3550 1800 30  0001 C CNN
+F 0 "#PWR6" H 3550 1800 30  0001 C CNN
 F 1 "GND" H 3550 1730 30  0001 C CNN
 F 2 "" H 3550 1800 60  0000 C CNN
@@
 $EndComp
 $Comp
-L GND #PWR05
+L GND #PWR3
 U 1 1 55011060
 P 1650 1800
-F 0 "#PWR05" H 1650 1800 30  0001 C CNN
+F 0 "#PWR3" H 1650 1800 30  0001 C CNN
 F 1 "GND" H 1650 1730 30  0001 C CNN
 F 2 "" H 1650 1800 60  0000 C CNN
@@
 $EndComp
 $Comp
-L GND #PWR06
+L GND #PWR8
 U 1 1 55280CC3
 P 3800 1150
-F 0 "#PWR06" H 3800 1150 30  0001 C CNN
+F 0 "#PWR8" H 3800 1150 30  0001 C CNN
 F 1 "GND" H 3800 1080 30  0001 C CNN
 F 2 "" H 3800 1150 60  0000 C CNN
@@
 VSense
 $Comp
-L +3.3V #PWR07
+L +3.3V #PWR10
 U 1 1 55280D8C
 P 4050 3800
-F 0 "#PWR07" H 4050 3760 30  0001 C CNN
+F 0 "#PWR10" H 4050 3760 30  0001 C CNN
 F 1 "+3.3V" H 4050 3910 30  0000 C CNN
 F 2 "" H 4050 3800 60  0000 C CNN
@@
 $EndComp
 $Comp
-L GND #PWR08
+L GND #PWR5
 U 1 1 55280D9B
 P 3300 4150
-F 0 "#PWR08" H 3300 4150 30  0001 C CNN
+F 0 "#PWR5" H 3300 4150 30  0001 C CNN
 F 1 "GND" H 3300 4080 30  0001 C CNN
 F 2 "" H 3300 4150 60  0000 C CNN
@@
 VBatt
 $Comp
-L GND #PWR09
+L GND #PWR12
 U 1 1 55281188
 P 7650 3850
-F 0 "#PWR09" H 7650 3850 30  0001 C CNN
+F 0 "#PWR12" H 7650 3850 30  0001 C CNN
 F 1 "GND" H 7650 3780 30  0001 C CNN
 F 2 "" H 7650 3850 60  0000 C CNN
@@
 I2C DAT
 $Comp
-L +3.3V #PWR010
+L +3.3V #PWR1
 U 1 1 552816BB
 P 1250 5150
-F 0 "#PWR010" H 1250 5110 30  0001 C CNN
+F 0 "#PWR1" H 1250 5110 30  0001 C CNN
 F 1 "+3.3V" H 1250 5260 30  0000 C CNN
 F 2 "" H 1250 5150 60  0000 C CNN
@@
 $EndComp
 $Comp
-L GND #PWR011
+L GND #PWR2
 U 1 1 55281865
 P 1250 7500
-F 0 "#PWR011" H 1250 7500 30  0001 C CNN
+F 0 "#PWR2" H 1250 7500 30  0001 C CNN
 F 1 "GND" H 1250 7430 30  0001 C CNN
 F 2 "" H 1250 7500 60  0000 C CNN
@@
 Reset
 $Comp
-L GND #PWR012
+L GND #PWR11
 U 1 1 55281D1D
 P 4500 6500
-F 0 "#PWR012" H 4500 6500 30  0001 C CNN
+F 0 "#PWR11" H 4500 6500 30  0001 C CNN
 F 1 "GND" H 4500 6430 30  0001 C CNN
 F 2 "" H 4500 6500 60  0000 C CNN
@@
 UART TX
 $Comp
-L GND #PWR013
+L GND #PWR16
 U 1 1 552825A2
 P 7950 6500
-F 0 "#PWR013" H 7950 6500 30  0001 C CNN
+F 0 "#PWR16" H 7950 6500 30  0001 C CNN
 F 1 "GND" H 7950 6430 30  0001 C CNN
 F 2 "" H 7950 6500 60  0000 C CNN
@@
 $EndComp
 $Comp
-L +3.3V #PWR014
+L +3.3V #PWR14
 U 1 1 552825B1
 P 7650 6500
-F 0 "#PWR014" H 7650 6460 30  0001 C CNN
+F 0 "#PWR14" H 7650 6460 30  0001 C CNN
 F 1 "+3.3V" H 7650 6610 30  0000 C CNN
 F 2 "" H 7650 6500 60  0000 C CNN
@@
 $EndComp
 $Comp
-L +3.3V #PWR015
+L +3.3V #PWR13
 U 1 1 55282851
 P 7650 6100
-F 0 "#PWR015" H 7650 6060 30  0001 C CNN
+F 0 "#PWR13" H 7650 6060 30  0001 C CNN
 F 1 "+3.3V" H 7650 6210 30  0000 C CNN
 F 2 "" H 7650 6100 60  0000 C CNN
@@
 $EndComp
 $Comp
-L GND #PWR016
+L GND #PWR20
 U 1 1 55282A83
 P 9750 1850
-F 0 "#PWR016" H 9750 1850 30  0001 C CNN
+F 0 "#PWR20" H 9750 1850 30  0001 C CNN
 F 1 "GND" H 9750 1780 30  0001 C CNN
 F 2 "" H 9750 1850 60  0000 C CNN
@@
 $EndComp
 $Comp
-L +3.3V #PWR017
+L +3.3V #PWR19
 U 1 1 55282A89
 P 9750 1750
-F 0 "#PWR017" H 9750 1710 30  0001 C CNN
+F 0 "#PWR19" H 9750 1710 30  0001 C CNN
 F 1 "+3.3V" H 9750 1860 30  0000 C CNN
 F 2 "" H 9750 1750 60  0000 C CNN
@@
 MOSI
 $Comp
-L GND #PWR018
+L GND #PWR23
 U 1 1 55282C20
 P 10200 6100
-F 0 "#PWR018" H 10200 6100 30  0001 C CNN
+F 0 "#PWR23" H 10200 6100 30  0001 C CNN
 F 1 "GND" H 10200 6030 30  0001 C CNN
 F 2 "" H 10200 6100 60  0000 C CNN
@@
 $EndComp
 $Comp
-L +3.3V #PWR019
+L +3.3V #PWR22
 U 1 1 55282C26
 P 10200 5900
-F 0 "#PWR019" H 10200 5860 30  0001 C CNN
+F 0 "#PWR22" H 10200 5860 30  0001 C CNN
 F 1 "+3.3V" H 10200 6010 30  0000 C CNN
 F 2 "" H 10200 5900 60  0000 C CNN
@@
 $EndComp
 $Comp
-L GND #PWR020
+L GND #PWR21
 U 1 1 55282D84
 P 10100 4300
-F 0 "#PWR020" H 10100 4300 30  0001 C CNN
+F 0 "#PWR21" H 10100 4300 30  0001 C CNN
 F 1 "GND" H 10100 4230 30  0001 C CNN
 F 2 "" H 10100 4300 60  0000 C CNN
@@
 $EndComp
 $Comp
-L +3.3V #PWR021
+L +3.3V #PWR24
 U 1 1 55282FA8
 P 10600 3400
-F 0 "#PWR021" H 10600 3360 30  0001 C CNN
+F 0 "#PWR24" H 10600 3360 30  0001 C CNN
 F 1 "+3.3V" H 10600 3510 30  0000 C CNN
 F 2 "" H 10600 3400 60  0000 C CNN
@@
 Rumble
 $Comp
-L GND #PWR022
+L GND #PWR17
 U 1 1 55283776
 P 8050 2000
-F 0 "#PWR022" H 8050 2000 30  0001 C CNN
+F 0 "#PWR17" H 8050 2000 30  0001 C CNN
 F 1 "GND" H 8050 1930 30  0001 C CNN
 F 2 "" H 8050 2000 60  0000 C CNN
@@
 $EndComp
 $Comp
-L GND #PWR023
+L GND #PWR15
 U 1 1 552837AD
 P 7800 1200
-F 0 "#PWR023" H 7800 1200 30  0001 C CNN
+F 0 "#PWR15" H 7800 1200 30  0001 C CNN
 F 1 "GND" H 7800 1130 30  0001 C CNN
 F 2 "" H 7800 1200 60  0000 C CNN
@@
 $EndComp
 $Comp
-L GND #PWR024
+L GND #PWR18
 U 1 1 5530A16F
 P 8350 6200
-F 0 "#PWR024" H 8350 6200 30  0001 C CNN
+F 0 "#PWR18" H 8350 6200 30  0001 C CNN
 F 1 "GND" H 8350 6130 30  0001 C CNN
 F 2 "" H 8350 6200 60  0000 C CNN
@@
 	1    0    0    -1
 $EndComp
-$Comp
-L JUMPER JP1
-U 1 1 5530A4A4
-P 3500 6950
-F 0 "JP1" H 3500 6850 60  0000 C CNN
-F 1 "JUMPER" H 3500 7050 60  0000 C CNN
-F 2 "" H 3500 6950 60  0000 C CNN
-F 3 "" H 3500 6950 60  0000 C CNN
-	1    3500 6950
-	-1   0    0    1
-$EndComp
 Connection ~ 2150 1550
 Wire Wire Line
@@
 Wire Wire Line
 	3800 6950 3750 6950
+$Comp
+L JUMPER JP1
+U 1 1 5530B17C
+P 3550 6950
+F 0 "JP1" H 3550 6850 60  0000 C CNN
+F 1 "JUMPER" H 3550 7050 60  0000 C CNN
+F 2 "~" H 3550 6950 60  0000 C CNN
+F 3 "~" H 3550 6950 60  0000 C CNN
+	1    3550 6950
+	1    0    0    -1
+$EndComp
 $EndSCHEMATC

Commit message: Quick Update #1 4/24
Parts:
- added R8: 220, ~, symbol R
Connections:
- net +3.3V: now also C3.1, D3.1 (A), U2.2 (OUT); no longer D3.2 (K)
- net GND: now also R8.2
- new net: D3.2 (K), R8.1
Changed lines of the file:
@@
 Sheet 1 1
 Title ""
-Date "17 apr 2015"
+Date "24 apr 2015"
 Rev ""
 Comp ""
@@
 VSense
 $Comp
-L +3.3V #PWR10
+L +3.3V #PWR11
 U 1 1 55280D8C
-P 4050 3800
-F 0 "#PWR10" H 4050 3760 30  0001 C CNN
-F 1 "+3.3V" H 4050 3910 30  0000 C CNN
-F 2 "" H 4050 3800 60  0000 C CNN
-F 3 "" H 4050 3800 60  0000 C CNN
-	1    4050 3800
-	-1   0    0    1
+P 4250 3300
+F 0 "#PWR11" H 4250 3260 30  0001 C CNN
+F 1 "+3.3V" H 4250 3410 30  0000 C CNN
+F 2 "" H 4250 3300 60  0000 C CNN
+F 3 "" H 4250 3300 60  0000 C CNN
+	1    4250 3300
+	0    1    1    0
 $EndComp
 $Comp
@@
 VBatt
 $Comp
-L GND #PWR12
+L GND #PWR13
 U 1 1 55281188
 P 7650 3850
-F 0 "#PWR12" H 7650 3850 30  0001 C CNN
+F 0 "#PWR13" H 7650 3850 30  0001 C CNN
 F 1 "GND" H 7650 3780 30  0001 C CNN
 F 2 "" H 7650 3850 60  0000 C CNN
@@
 Reset
 $Comp
-L GND #PWR11
+L GND #PWR12
 U 1 1 55281D1D
 P 4500 6500
-F 0 "#PWR11" H 4500 6500 30  0001 C CNN
+F 0 "#PWR12" H 4500 6500 30  0001 C CNN
 F 1 "GND" H 4500 6430 30  0001 C CNN
 F 2 "" H 4500 6500 60  0000 C CNN
@@
 UART TX
 $Comp
-L GND #PWR16
+L GND #PWR17
 U 1 1 552825A2
 P 7950 6500
-F 0 "#PWR16" H 7950 6500 30  0001 C CNN
+F 0 "#PWR17" H 7950 6500 30  0001 C CNN
 F 1 "GND" H 7950 6430 30  0001 C CNN
 F 2 "" H 7950 6500 60  0000 C CNN
@@
 $EndComp
 $Comp
-L +3.3V #PWR14
+L +3.3V #PWR15
 U 1 1 552825B1
 P 7650 6500
-F 0 "#PWR14" H 7650 6460 30  0001 C CNN
+F 0 "#PWR15" H 7650 6460 30  0001 C CNN
 F 1 "+3.3V" H 7650 6610 30  0000 C CNN
 F 2 "" H 7650 6500 60  0000 C CNN
@@
 $EndComp
 $Comp
-L +3.3V #PWR13
+L +3.3V #PWR14
 U 1 1 55282851
 P 7650 6100
-F 0 "#PWR13" H 7650 6060 30  0001 C CNN
+F 0 "#PWR14" H 7650 6060 30  0001 C CNN
 F 1 "+3.3V" H 7650 6210 30  0000 C CNN
 F 2 "" H 7650 6100 60  0000 C CNN
@@
 $EndComp
 $Comp
-L GND #PWR20
+L GND #PWR21
 U 1 1 55282A83
 P 9750 1850
-F 0 "#PWR20" H 9750 1850 30  0001 C CNN
+F 0 "#PWR21" H 9750 1850 30  0001 C CNN
 F 1 "GND" H 9750 1780 30  0001 C CNN
 F 2 "" H 9750 1850 60  0000 C CNN
@@
 $EndComp
 $Comp
-L +3.3V #PWR19
+L +3.3V #PWR20
 U 1 1 55282A89
 P 9750 1750
-F 0 "#PWR19" H 9750 1710 30  0001 C CNN
+F 0 "#PWR20" H 9750 1710 30  0001 C CNN
 F 1 "+3.3V" H 9750 1860 30  0000 C CNN
 F 2 "" H 9750 1750 60  0000 C CNN
@@
 MOSI
 $Comp
-L GND #PWR23
+L GND #PWR24
 U 1 1 55282C20
 P 10200 6100
-F 0 "#PWR23" H 10200 6100 30  0001 C CNN
+F 0 "#PWR24" H 10200 6100 30  0001 C CNN
 F 1 "GND" H 10200 6030 30  0001 C CNN
 F 2 "" H 10200 6100 60  0000 C CNN
@@
 $EndComp
 $Comp
-L +3.3V #PWR22
+L +3.3V #PWR23
 U 1 1 55282C26
 P 10200 5900
-F 0 "#PWR22" H 10200 5860 30  0001 C CNN
+F 0 "#PWR23" H 10200 5860 30  0001 C CNN
 F 1 "+3.3V" H 10200 6010 30  0000 C CNN
 F 2 "" H 10200 5900 60  0000 C CNN
@@
 $EndComp
 $Comp
-L GND #PWR21
+L GND #PWR22
 U 1 1 55282D84
 P 10100 4300
-F 0 "#PWR21" H 10100 4300 30  0001 C CNN
+F 0 "#PWR22" H 10100 4300 30  0001 C CNN
 F 1 "GND" H 10100 4230 30  0001 C CNN
 F 2 "" H 10100 4300 60  0000 C CNN
@@
 $EndComp
 $Comp
-L +3.3V #PWR24
+L +3.3V #PWR25
 U 1 1 55282FA8
 P 10600 3400
-F 0 "#PWR24" H 10600 3360 30  0001 C CNN
+F 0 "#PWR25" H 10600 3360 30  0001 C CNN
 F 1 "+3.3V" H 10600 3510 30  0000 C CNN
 F 2 "" H 10600 3400 60  0000 C CNN
@@
 Rumble
 $Comp
-L GND #PWR17
+L GND #PWR18
 U 1 1 55283776
 P 8050 2000
-F 0 "#PWR17" H 8050 2000 30  0001 C CNN
+F 0 "#PWR18" H 8050 2000 30  0001 C CNN
 F 1 "GND" H 8050 1930 30  0001 C CNN
 F 2 "" H 8050 2000 60  0000 C CNN
@@
 $EndComp
 $Comp
-L GND #PWR15
+L GND #PWR16
 U 1 1 552837AD
 P 7800 1200
-F 0 "#PWR15" H 7800 1200 30  0001 C CNN
+F 0 "#PWR16" H 7800 1200 30  0001 C CNN
 F 1 "GND" H 7800 1130 30  0001 C CNN
 F 2 "" H 7800 1200 60  0000 C CNN
@@
 $EndComp
 $Comp
-L GND #PWR18
+L GND #PWR19
 U 1 1 5530A16F
 P 8350 6200
-F 0 "#PWR18" H 8350 6200 30  0001 C CNN
+F 0 "#PWR19" H 8350 6200 30  0001 C CNN
 F 1 "GND" H 8350 6130 30  0001 C CNN
 F 2 "" H 8350 6200 60  0000 C CNN
@@
 	3700 3500 3700 3300
 Wire Wire Line
-	3700 3300 4050 3300
+	3700 3300 4250 3300
 Wire Wire Line
 	3700 3900 3700 4000
@@
 Wire Wire Line
 	2000 3300 2100 3300
-Wire Wire Line
-	4050 3700 4050 3800
 Wire Notes Line
 	500  4550 5600 4550
@@
 	1    0    0    -1
 $EndComp
+Connection ~ 4050 3300
+$Comp
+L R R8
+U 1 1 5539BEA2
+P 4050 3950
+F 0 "R8" V 4130 3950 40  0000 C CNN
+F 1 "220" V 4057 3951 40  0000 C CNN
+F 2 "~" V 3980 3950 30  0000 C CNN
+F 3 "~" H 4050 3950 30  0000 C CNN
+	1    4050 3950
+	1    0    0    -1
+$EndComp
+$Comp
+L GND #PWR10
+U 1 1 5539BEBB
+P 4050 4200
+F 0 "#PWR10" H 4050 4200 30  0001 C CNN
+F 1 "GND" H 4050 4130 30  0001 C CNN
+F 2 "" H 4050 4200 60  0000 C CNN
+F 3 "" H 4050 4200 60  0000 C CNN
+	1    4050 4200
+	1    0    0    -1
+$EndComp

Commit message: Quick Update #2 4/24
Parts:
- removed D1: LED, ~, symbol LED
Connections:
- net VBatt: now also R2.1, U2.3 (IN)
- net VSense: no longer R3.1
Changed lines of the file:
@@
 Text GLabel 2000 3300 0    60   Input ~ 0
 VBatt
-Text GLabel 2600 4000 0    60   Output ~ 0
+Text GLabel 2750 4050 3    60   Output ~ 0
 VSense
 $Comp
@@
 Text Notes 7650 2800 2    118  ~ 0
 AlphaNumeric Display
-$Comp
-L LED D1
-U 1 1 5528124B
-P 2300 3300
-F 0 "D1" H 2300 3400 50  0000 C CNN
-F 1 "LED" H 2300 3200 50  0000 C CNN
-F 2 "~" H 2300 3300 60  0000 C CNN
-F 3 "~" H 2300 3300 60  0000 C CNN
-	1    2300 3300
-	1    0    0    -1
-$EndComp
 $Comp
 L LED D3
@@
 	5600 500  5600 7800
 Wire Wire Line
-	2500 3300 2900 3300
+	2000 3300 2900 3300
 Wire Wire Line
 	2750 3400 2750 3300
 Connection ~ 2750 3300
 Wire Wire Line
-	2750 3900 2750 4000
+	2750 3900 2750 4050
 Connection ~ 2750 4000
 Wire Wire Line
@@
 Connection ~ 3300 4000
 Wire Wire Line
-	2800 4000 2600 4000
-Wire Wire Line
 	3700 3500 3700 3300
 Wire Wire Line
@@
 Wire Wire Line
 	7400 4000 7650 4000
-Wire Wire Line
-	2000 3300 2100 3300
 Wire Notes Line
 	500  4550 5600 4550
