File: KiCad/Player-Health/Player-Health.sch (KiCad schematic (older format))
At the start: 34 parts, among them IC1 ATMEGA328-P, J1 MICRO_USB, M1 RUMBLE, P1 2P_CGRID_M, P2 6pM CGrid, P3 6pM Header, P4 8pF Header, Q1 NPN, U1 MCP73831, U2 LM1084IT-3.3/NOPB, U3 14SLED, U4 ESP8266, X1 CRYSTAL

Commit message: Quick Update 5/1
Parts:
- added C?: 4.7 uF, ~, symbol C
Connections:
- net LED B: no longer P2.5
- net LED G: no longer P2.4
- net LED R: no longer P2.6
- net VSense: now also C?.2; no longer R2.2
- net at R3.1: now also R2.2, C?.1
Other:
- moved on the sheet: C3, D3, P2, R2, R3, R8, U2
Changed lines of the file:
@@
 Sheet 1 1
 Title ""
-Date "24 apr 2015"
+Date "1 may 2015"
 Rev ""
 Comp ""
@@
 L LM1084IT-3.3/NOPB U2
 U 1 1 5501240B
-P 3300 3350
-F 0 "U2" H 3500 3150 40  0000 C CNN
-F 1 "LM1084IT-3.3/NOPB" H 3000 3550 40  0000 L CNN
-F 2 "TO-220" H 3300 3450 30  0000 C CIN
-F 3 "~" H 3300 3350 60  0000 C CNN
-	1    3300 3350
+P 3150 3200
+F 0 "U2" H 3350 3000 40  0000 C CNN
+F 1 "LM1084IT-3.3/NOPB" H 2850 3400 40  0000 L CNN
+F 2 "TO-220" H 3150 3300 30  0000 C CIN
+F 3 "~" H 3150 3200 60  0000 C CNN
+	1    3150 3200
 	1    0    0    -1
 $EndComp
@@
 L R R2
 U 1 1 55280D5E
-P 2750 3650
-F 0 "R2" V 2830 3650 40  0000 C CNN
-F 1 "10k" V 2757 3651 40  0000 C CNN
-F 2 "~" V 2680 3650 30  0000 C CNN
-F 3 "~" H 2750 3650 30  0000 C CNN
-	1    2750 3650
+P 2600 3500
+F 0 "R2" V 2680 3500 40  0000 C CNN
+F 1 "10k" V 2607 3501 40  0000 C CNN
+F 2 "~" V 2530 3500 30  0000 C CNN
+F 3 "~" H 2600 3500 30  0000 C CNN
+	1    2600 3500
 	1    0    0    -1
 $EndComp
@@
 L R R3
 U 1 1 55280D64
-P 3050 4000
-F 0 "R3" V 3130 4000 40  0000 C CNN
-F 1 "10k" V 3057 4001 40  0000 C CNN
-F 2 "~" V 2980 4000 30  0000 C CNN
-F 3 "~" H 3050 4000 30  0000 C CNN
-	1    3050 4000
+P 2900 3850
+F 0 "R3" V 2980 3850 40  0000 C CNN
+F 1 "10k" V 2907 3851 40  0000 C CNN
+F 2 "~" V 2830 3850 30  0000 C CNN
+F 3 "~" H 2900 3850 30  0000 C CNN
+	1    2900 3850
 	0    -1   -1   0
 $EndComp
@@
 L C C3
 U 1 1 55280D6C
-P 3700 3700
-F 0 "C3" H 3700 3800 40  0000 L CNN
-F 1 "100uF" H 3706 3615 40  0000 L CNN
-F 2 "~" H 3738 3550 30  0000 C CNN
-F 3 "~" H 3700 3700 60  0000 C CNN
-	1    3700 3700
-	1    0    0    -1
-$EndComp
-Text GLabel 2000 3300 0    60   Input ~ 0
+P 3550 3550
+F 0 "C3" H 3550 3650 40  0000 L CNN
+F 1 "100uF" H 3556 3465 40  0000 L CNN
+F 2 "~" H 3588 3400 30  0000 C CNN
+F 3 "~" H 3550 3550 60  0000 C CNN
+	1    3550 3550
+	1    0    0    -1
+$EndComp
+Text GLabel 1850 3150 0    60   Input ~ 0
 VBatt
-Text GLabel 2750 4050 3    60   Output ~ 0
+Text GLabel 2750 4300 2    60   Output ~ 0
 VSense
 $Comp
 L +3.3V #PWR11
 U 1 1 55280D8C
-P 4250 3300
-F 0 "#PWR11" H 4250 3260 30  0001 C CNN
-F 1 "+3.3V" H 4250 3410 30  0000 C CNN
-F 2 "" H 4250 3300 60  0000 C CNN
-F 3 "" H 4250 3300 60  0000 C CNN
-	1    4250 3300
+P 4100 3150
+F 0 "#PWR11" H 4100 3110 30  0001 C CNN
+F 1 "+3.3V" H 4100 3260 30  0000 C CNN
+F 2 "" H 4100 3150 60  0000 C CNN
+F 3 "" H 4100 3150 60  0000 C CNN
+	1    4100 3150
 	0    1    1    0
 $EndComp
@@
 L GND #PWR5
 U 1 1 55280D9B
-P 3300 4150
-F 0 "#PWR5" H 3300 4150 30  0001 C CNN
-F 1 "GND" H 3300 4080 30  0001 C CNN
-F 2 "" H 3300 4150 60  0000 C CNN
-F 3 "" H 3300 4150 60  0000 C CNN
-	1    3300 4150
+P 3150 4000
+F 0 "#PWR5" H 3150 4000 30  0001 C CNN
+F 1 "GND" H 3150 3930 30  0001 C CNN
+F 2 "" H 3150 4000 60  0000 C CNN
+F 3 "" H 3150 4000 60  0000 C CNN
+	1    3150 4000
 	1    0    0    -1
 $EndComp
@@
 L LED D3
 U 1 1 552812BB
-P 4050 3500
-F 0 "D3" H 4050 3600 50  0000 C CNN
-F 1 "LED" H 4050 3400 50  0000 C CNN
-F 2 "~" H 4050 3500 60  0000 C CNN
-F 3 "~" H 4050 3500 60  0000 C CNN
-	1    4050 3500
+P 3900 3350
+F 0 "D3" H 3900 3450 50  0000 C CNN
+F 1 "LED" H 3900 3250 50  0000 C CNN
+F 2 "~" H 3900 3350 60  0000 C CNN
+F 3 "~" H 3900 3350 60  0000 C CNN
+	1    3900 3350
 	0    1    1    0
 $EndComp
@@
 L CONN_6 P2
 U 1 1 55282A50
-P 9400 1600
-F 0 "P2" V 9350 1600 60  0000 C CNN
-F 1 "6pM CGrid" V 9450 1600 60  0000 C CNN
-F 2 "" H 9400 1600 60  0000 C CNN
-F 3 "" H 9400 1600 60  0000 C CNN
-	1    9400 1600
+P 9150 1850
+F 0 "P2" V 9100 1850 60  0000 C CNN
+F 1 "6pM CGrid" V 9200 1850 60  0000 C CNN
+F 2 "" H 9150 1850 60  0000 C CNN
+F 3 "" H 9150 1850 60  0000 C CNN
+	1    9150 1850
 	-1   0    0    1
 $EndComp
@@
 L GND #PWR21
 U 1 1 55282A83
-P 9750 1850
-F 0 "#PWR21" H 9750 1850 30  0001 C CNN
-F 1 "GND" H 9750 1780 30  0001 C CNN
-F 2 "" H 9750 1850 60  0000 C CNN
-F 3 "" H 9750 1850 60  0000 C CNN
-	1    9750 1850
+P 9500 2100
+F 0 "#PWR21" H 9500 2100 30  0001 C CNN
+F 1 "GND" H 9500 2030 30  0001 C CNN
+F 2 "" H 9500 2100 60  0000 C CNN
+F 3 "" H 9500 2100 60  0000 C CNN
+	1    9500 2100
 	0    -1   -1   0
 $EndComp
@@
 L +3.3V #PWR20
 U 1 1 55282A89
-P 9750 1750
-F 0 "#PWR20" H 9750 1710 30  0001 C CNN
-F 1 "+3.3V" H 9750 1860 30  0000 C CNN
-F 2 "" H 9750 1750 60  0000 C CNN
-F 3 "" H 9750 1750 60  0000 C CNN
-	1    9750 1750
+P 9500 2000
+F 0 "#PWR20" H 9500 1960 30  0001 C CNN
+F 1 "+3.3V" H 9500 2110 30  0000 C CNN
+F 2 "" H 9500 2000 60  0000 C CNN
+F 3 "" H 9500 2000 60  0000 C CNN
+	1    9500 2000
 	0    1    1    0
 $EndComp
-Text GLabel 10100 1650 2    59   BiDi ~ 0
+Text GLabel 10250 1900 2    59   BiDi ~ 0
 IR Sense
-Text GLabel 10100 1450 2    59   BiDi ~ 0
+Text GLabel 10600 1450 1    59   BiDi ~ 0
 LED B
-Text GLabel 9750 1350 2    59   BiDi ~ 0
+Text GLabel 10400 1450 1    59   BiDi ~ 0
 LED R
-Text GLabel 9750 1550 2    59   BiDi ~ 0
+Text GLabel 10800 1450 1    59   BiDi ~ 0
 LED G
 Text Notes 8800 700  0    118  ~ 0
@@
 	5600 500  5600 7800
 Wire Wire Line
-	2000 3300 2900 3300
-Wire Wire Line
-	2750 3400 2750 3300
-Connection ~ 2750 3300
-Wire Wire Line
-	2750 3900 2750 4050
-Connection ~ 2750 4000
-Wire Wire Line
-	3300 3600 3300 4150
-Connection ~ 3300 4000
-Wire Wire Line
-	3700 3500 3700 3300
-Wire Wire Line
-	3700 3300 4250 3300
-Wire Wire Line
-	3700 3900 3700 4000
-Wire Wire Line
-	3700 4000 3300 4000
+	1850 3150 2750 3150
+Wire Wire Line
+	2600 3250 2600 3150
+Connection ~ 2600 3150
+Wire Wire Line
+	2600 3750 2600 3900
+Connection ~ 2600 3850
+Wire Wire Line
+	3150 3450 3150 4000
+Connection ~ 3150 3850
+Wire Wire Line
+	3550 3350 3550 3150
+Wire Wire Line
+	3550 3150 4100 3150
+Wire Wire Line
+	3550 3750 3550 3850
+Wire Wire Line
+	3550 3850 3150 3850
 Wire Wire Line
 	7650 3550 7400 3550
@@
 	7800 6200 7650 6200
 Wire Wire Line
-	9750 1650 10100 1650
-Wire Wire Line
-	10100 1450 9750 1450
+	9500 1900 10250 1900
 Wire Wire Line
 	10200 6400 9900 6400
@@
 	1    0    0    -1
 $EndComp
-Connection ~ 4050 3300
+Connection ~ 3900 3150
 $Comp
 L R R8
 U 1 1 5539BEA2
-P 4050 3950
-F 0 "R8" V 4130 3950 40  0000 C CNN
-F 1 "220" V 4057 3951 40  0000 C CNN
-F 2 "~" V 3980 3950 30  0000 C CNN
-F 3 "~" H 4050 3950 30  0000 C CNN
-	1    4050 3950
+P 3900 3800
+F 0 "R8" V 3980 3800 40  0000 C CNN
+F 1 "220" V 3907 3801 40  0000 C CNN
+F 2 "~" V 3830 3800 30  0000 C CNN
+F 3 "~" H 3900 3800 30  0000 C CNN
+	1    3900 3800
 	1    0    0    -1
 $EndComp
@@
 L GND #PWR10
 U 1 1 5539BEBB
-P 4050 4200
-F 0 "#PWR10" H 4050 4200 30  0001 C CNN
-F 1 "GND" H 4050 4130 30  0001 C CNN
-F 2 "" H 4050 4200 60  0000 C CNN
-F 3 "" H 4050 4200 60  0000 C CNN
-	1    4050 4200
-	1    0    0    -1
-$EndComp
+P 3900 4050
+F 0 "#PWR10" H 3900 4050 30  0001 C CNN
+F 1 "GND" H 3900 3980 30  0001 C CNN
+F 2 "" H 3900 4050 60  0000 C CNN
+F 3 "" H 3900 4050 60  0000 C CNN
+	1    3900 4050
+	1    0    0    -1
+$EndComp
+Wire Wire Line
+	2650 3850 2600 3850
+$Comp
+L C C?
+U 1 1 5542E5DC
+P 2600 4100
+F 0 "C?" H 2600 4200 40  0000 L CNN
+F 1 "4.7 uF" H 2606 4015 40  0000 L CNN
+F 2 "~" H 2638 3950 30  0000 C CNN
+F 3 "~" H 2600 4100 60  0000 C CNN
+	1    2600 4100
+	1    0    0    -1
+$EndComp
+Wire Wire Line
+	2750 4300 2600 4300
+Wire Notes Line
+	9450 1350 9450 2100
+Wire Notes Line
+	9450 2100 10900 2100
+Wire Notes Line
+	10900 2100 10900 1000
+Wire Notes Line
+	10900 1000 9600 1000
 $EndSCHEMATC

Commit message: Quick Update #2 5/1
Night night
Parts:
- added Q? (x3): NPN, ~, symbol NPN
Connections:
- net GND: now also C?.2
- net VSense: now also C?.1, R2.2, R3.1; no longer C?.2
Other:
- moved on the sheet: C?
Changed lines of the file:
@@
 Text GLabel 1850 3150 0    60   Input ~ 0
 VBatt
-Text GLabel 2750 4300 2    60   Output ~ 0
+Text GLabel 2600 3950 3    60   Output ~ 0
 VSense
 $Comp
@@
 $EndComp
 Wire Wire Line
-	2650 3850 2600 3850
+	2200 3850 2650 3850
 $Comp
 L C C?
 U 1 1 5542E5DC
-P 2600 4100
-F 0 "C?" H 2600 4200 40  0000 L CNN
-F 1 "4.7 uF" H 2606 4015 40  0000 L CNN
-F 2 "~" H 2638 3950 30  0000 C CNN
-F 3 "~" H 2600 4100 60  0000 C CNN
-	1    2600 4100
-	1    0    0    -1
-$EndComp
-Wire Wire Line
-	2750 4300 2600 4300
+P 2200 4050
+F 0 "C?" H 2200 4150 40  0000 L CNN
+F 1 "4.7 uF" H 2206 3965 40  0000 L CNN
+F 2 "~" H 2238 3900 30  0000 C CNN
+F 3 "~" H 2200 4050 60  0000 C CNN
+	1    2200 4050
+	1    0    0    -1
+$EndComp
 Wire Notes Line
 	9450 1350 9450 2100
@@
 Wire Notes Line
 	10900 1000 9600 1000
+Wire Wire Line
+	2600 3850 2600 3950
+$Comp
+L GND #PWR?
+U 1 1 55430D54
+P 2200 4300
+F 0 "#PWR?" H 2200 4300 30  0001 C CNN
+F 1 "GND" H 2200 4230 30  0001 C CNN
+F 2 "" H 2200 4300 60  0000 C CNN
+F 3 "" H 2200 4300 60  0000 C CNN
+	1    2200 4300
+	1    0    0    -1
+$EndComp
+Wire Wire Line
+	2200 4300 2200 4250
+$Comp
+L NPN Q?
+U 1 1 554310E6
+P 9900 1300
+F 0 "Q?" H 9900 1150 50  0000 R CNN
+F 1 "NPN" H 9900 1450 50  0000 R CNN
+F 2 "~" H 9900 1300 60  0000 C CNN
+F 3 "~" H 9900 1300 60  0000 C CNN
+	1    9900 1300
+	0    1    1    0
+$EndComp
+$Comp
+L NPN Q?
+U 1 1 554310F6
+P 10100 1700
+F 0 "Q?" H 10100 1550 50  0000 R CNN
+F 1 "NPN" H 10100 1850 50  0000 R CNN
+F 2 "~" H 10100 1700 60  0000 C CNN
+F 3 "~" H 10100 1700 60  0000 C CNN
+	1    10100 1700
+	0    1    1    0
+$EndComp
+$Comp
+L NPN Q?
+U 1 1 554310FC
+P 9250 1250
+F 0 "Q?" H 9250 1100 50  0000 R CNN
+F 1 "NPN" H 9250 1400 50  0000 R CNN
+F 2 "~" H 9250 1250 60  0000 C CNN
+F 3 "~" H 9250 1250 60  0000 C CNN
+	1    9250 1250
+	0    1    1    0
+$EndComp
 $EndSCHEMATC

Commit message: Quick Update #3 5/1
Potential last changes before ordering ir receiver and player boards
Parts:
- gave numbers to parts that had none: 4
Connections:
- net LED B: now also Q3.2 (B)
- net LED G: now also Q4.2 (B)
- net LED R: now also Q2.2 (B)
- net VBatt: now also Q2.3 (C), Q3.3 (C), Q4.3 (C)
- net at P2.4: now also Q4.1 (E)
- net at P2.5: now also Q3.1 (E)
- net at P2.6: now also Q2.1 (E)
Other:
- moved on the sheet: P2, Q2, Q3, Q4
Changed lines of the file:
@@
 $EndComp
 $Comp
-L GND #PWR4
+L GND #PWR01
 U 1 1 5501101E
 P 1850 2050
-F 0 "#PWR4" H 1850 2050 30  0001 C CNN
+F 0 "#PWR01" H 1850 2050 30  0001 C CNN
 F 1 "GND" H 1850 1980 30  0001 C CNN
 F 2 "" H 1850 2050 60  0000 C CNN
@@
 $EndComp
 $Comp
-L GND #PWR9
+L GND #PWR02
 U 1 1 55011447
 P 3950 2300
-F 0 "#PWR9" H 3950 2300 30  0001 C CNN
+F 0 "#PWR02" H 3950 2300 30  0001 C CNN
 F 1 "GND" H 3950 2230 30  0001 C CNN
 F 2 "" H 3950 2300 60  0000 C CNN
@@
 $EndComp
 $Comp
-L GND #PWR7
+L GND #PWR03
 U 1 1 550112D9
 P 3700 2300
-F 0 "#PWR7" H 3700 2300 30  0001 C CNN
+F 0 "#PWR03" H 3700 2300 30  0001 C CNN
 F 1 "GND" H 3700 2230 30  0001 C CNN
 F 2 "" H 3700 2300 60  0000 C CNN
@@
 $EndComp
 $Comp
-L GND #PWR6
+L GND #PWR04
 U 1 1 5501126E
 P 3550 1800
-F 0 "#PWR6" H 3550 1800 30  0001 C CNN
+F 0 "#PWR04" H 3550 1800 30  0001 C CNN
 F 1 "GND" H 3550 1730 30  0001 C CNN
 F 2 "" H 3550 1800 60  0000 C CNN
@@
 $EndComp
 $Comp
-L GND #PWR3
+L GND #PWR05
 U 1 1 55011060
 P 1650 1800
-F 0 "#PWR3" H 1650 1800 30  0001 C CNN
+F 0 "#PWR05" H 1650 1800 30  0001 C CNN
 F 1 "GND" H 1650 1730 30  0001 C CNN
 F 2 "" H 1650 1800 60  0000 C CNN
@@
 $EndComp
 $Comp
-L GND #PWR8
+L GND #PWR06
 U 1 1 55280CC3
 P 3800 1150
-F 0 "#PWR8" H 3800 1150 30  0001 C CNN
+F 0 "#PWR06" H 3800 1150 30  0001 C CNN
 F 1 "GND" H 3800 1080 30  0001 C CNN
 F 2 "" H 3800 1150 60  0000 C CNN
@@
 VSense
 $Comp
-L +3.3V #PWR11
+L +3.3V #PWR07
 U 1 1 55280D8C
 P 4100 3150
-F 0 "#PWR11" H 4100 3110 30  0001 C CNN
+F 0 "#PWR07" H 4100 3110 30  0001 C CNN
 F 1 "+3.3V" H 4100 3260 30  0000 C CNN
 F 2 "" H 4100 3150 60  0000 C CNN
@@
 $EndComp
 $Comp
-L GND #PWR5
+L GND #PWR08
 U 1 1 55280D9B
 P 3150 4000
-F 0 "#PWR5" H 3150 4000 30  0001 C CNN
+F 0 "#PWR08" H 3150 4000 30  0001 C CNN
 F 1 "GND" H 3150 3930 30  0001 C CNN
 F 2 "" H 3150 4000 60  0000 C CNN
@@
 VBatt
 $Comp
-L GND #PWR13
+L GND #PWR09
 U 1 1 55281188
 P 7650 3850
-F 0 "#PWR13" H 7650 3850 30  0001 C CNN
+F 0 "#PWR09" H 7650 3850 30  0001 C CNN
 F 1 "GND" H 7650 3780 30  0001 C CNN
 F 2 "" H 7650 3850 60  0000 C CNN
@@
 I2C DAT
 $Comp
-L +3.3V #PWR1
+L +3.3V #PWR010
 U 1 1 552816BB
 P 1250 5150
-F 0 "#PWR1" H 1250 5110 30  0001 C CNN
+F 0 "#PWR010" H 1250 5110 30  0001 C CNN
 F 1 "+3.3V" H 1250 5260 30  0000 C CNN
 F 2 "" H 1250 5150 60  0000 C CNN
@@
 $EndComp
 $Comp
-L GND #PWR2
+L GND #PWR011
 U 1 1 55281865
 P 1250 7500
-F 0 "#PWR2" H 1250 7500 30  0001 C CNN
+F 0 "#PWR011" H 1250 7500 30  0001 C CNN
 F 1 "GND" H 1250 7430 30  0001 C CNN
 F 2 "" H 1250 7500 60  0000 C CNN
@@
 Reset
 $Comp
-L GND #PWR12
+L GND #PWR012
 U 1 1 55281D1D
 P 4500 6500
-F 0 "#PWR12" H 4500 6500 30  0001 C CNN
+F 0 "#PWR012" H 4500 6500 30  0001 C CNN
 F 1 "GND" H 4500 6430 30  0001 C CNN
 F 2 "" H 4500 6500 60  0000 C CNN
@@
 UART TX
 $Comp
-L GND #PWR17
+L GND #PWR013
 U 1 1 552825A2
 P 7950 6500
-F 0 "#PWR17" H 7950 6500 30  0001 C CNN
+F 0 "#PWR013" H 7950 6500 30  0001 C CNN
 F 1 "GND" H 7950 6430 30  0001 C CNN
 F 2 "" H 7950 6500 60  0000 C CNN
@@
 $EndComp
 $Comp
-L +3.3V #PWR15
+L +3.3V #PWR014
 U 1 1 552825B1
 P 7650 6500
-F 0 "#PWR15" H 7650 6460 30  0001 C CNN
+F 0 "#PWR014" H 7650 6460 30  0001 C CNN
 F 1 "+3.3V" H 7650 6610 30  0000 C CNN
 F 2 "" H 7650 6500 60  0000 C CNN
@@
 $EndComp
 $Comp
-L +3.3V #PWR14
+L +3.3V #PWR015
 U 1 1 55282851
 P 7650 6100
-F 0 "#PWR14" H 7650 6060 30  0001 C CNN
+F 0 "#PWR015" H 7650 6060 30  0001 C CNN
 F 1 "+3.3V" H 7650 6210 30  0000 C CNN
 F 2 "" H 7650 6100 60  0000 C CNN
@@
 L CONN_6 P2
 U 1 1 55282A50
-P 9150 1850
-F 0 "P2" V 9100 1850 60  0000 C CNN
-F 1 "6pM CGrid" V 9200 1850 60  0000 C CNN
-F 2 "" H 9150 1850 60  0000 C CNN
-F 3 "" H 9150 1850 60  0000 C CNN
-	1    9150 1850
+P 9000 1900
+F 0 "P2" V 8950 1900 60  0000 C CNN
+F 1 "6pM CGrid" V 9050 1900 60  0000 C CNN
+F 2 "" H 9000 1900 60  0000 C CNN
+F 3 "" H 9000 1900 60  0000 C CNN
+	1    9000 1900
 	-1   0    0    1
 $EndComp
 $Comp
-L GND #PWR21
+L GND #PWR016
 U 1 1 55282A83
-P 9500 2100
-F 0 "#PWR21" H 9500 2100 30  0001 C CNN
-F 1 "GND" H 9500 2030 30  0001 C CNN
-F 2 "" H 9500 2100 60  0000 C CNN
-F 3 "" H 9500 2100 60  0000 C CNN
-	1    9500 2100
-	0    -1   -1   0
-$EndComp
-$Comp
-L +3.3V #PWR20
+P 9350 2150
+F 0 "#PWR016" H 9350 2150 30  0001 C CNN
+F 1 "GND" H 9350 2080 30  0001 C CNN
+F 2 "" H 9350 2150 60  0000 C CNN
+F 3 "" H 9350 2150 60  0000 C CNN
+	1    9350 2150
+	0    -1   -1   0
+$EndComp
+$Comp
+L +3.3V #PWR017
 U 1 1 55282A89
-P 9500 2000
-F 0 "#PWR20" H 9500 1960 30  0001 C CNN
-F 1 "+3.3V" H 9500 2110 30  0000 C CNN
-F 2 "" H 9500 2000 60  0000 C CNN
-F 3 "" H 9500 2000 60  0000 C CNN
-	1    9500 2000
-	0    1    1    0
-$EndComp
-Text GLabel 10250 1900 2    59   BiDi ~ 0
+P 9350 2050
+F 0 "#PWR017" H 9350 2010 30  0001 C CNN
+F 1 "+3.3V" H 9350 2160 30  0000 C CNN
+F 2 "" H 9350 2050 60  0000 C CNN
+F 3 "" H 9350 2050 60  0000 C CNN
+	1    9350 2050
+	0    1    1    0
+$EndComp
+Text GLabel 10650 1950 2    59   BiDi ~ 0
 IR Sense
-Text GLabel 10600 1450 1    59   BiDi ~ 0
+Text GLabel 10000 1450 1    59   BiDi ~ 0
 LED B
-Text GLabel 10400 1450 1    59   BiDi ~ 0
+Text GLabel 9550 1350 1    59   BiDi ~ 0
 LED R
-Text GLabel 10800 1450 1    59   BiDi ~ 0
+Text GLabel 10450 1550 1    59   BiDi ~ 0
 LED G
 Text Notes 8800 700  0    118  ~ 0
@@
 MOSI
 $Comp
-L GND #PWR24
+L GND #PWR018
 U 1 1 55282C20
 P 10200 6100
-F 0 "#PWR24" H 10200 6100 30  0001 C CNN
+F 0 "#PWR018" H 10200 6100 30  0001 C CNN
 F 1 "GND" H 10200 6030 30  0001 C CNN
 F 2 "" H 10200 6100 60  0000 C CNN
@@
 $EndComp
 $Comp
-L +3.3V #PWR23
+L +3.3V #PWR019
 U 1 1 55282C26
 P 10200 5900
-F 0 "#PWR23" H 10200 5860 30  0001 C CNN
+F 0 "#PWR019" H 10200 5860 30  0001 C CNN
 F 1 "+3.3V" H 10200 6010 30  0000 C CNN
 F 2 "" H 10200 5900 60  0000 C CNN
@@
 $EndComp
 $Comp
-L GND #PWR22
+L GND #PWR020
 U 1 1 55282D84
 P 10100 4300
-F 0 "#PWR22" H 10100 4300 30  0001 C CNN
+F 0 "#PWR020" H 10100 4300 30  0001 C CNN
 F 1 "GND" H 10100 4230 30  0001 C CNN
 F 2 "" H 10100 4300 60  0000 C CNN
@@
 $EndComp
 $Comp
-L +3.3V #PWR25
+L +3.3V #PWR021
 U 1 1 55282FA8
 P 10600 3400
-F 0 "#PWR25" H 10600 3360 30  0001 C CNN
+F 0 "#PWR021" H 10600 3360 30  0001 C CNN
 F 1 "+3.3V" H 10600 3510 30  0000 C CNN
 F 2 "" H 10600 3400 60  0000 C CNN
@@
 Rumble
 $Comp
-L GND #PWR18
+L GND #PWR022
 U 1 1 55283776
 P 8050 2000
-F 0 "#PWR18" H 8050 2000 30  0001 C CNN
+F 0 "#PWR022" H 8050 2000 30  0001 C CNN
 F 1 "GND" H 8050 1930 30  0001 C CNN
 F 2 "" H 8050 2000 60  0000 C CNN
@@
 $EndComp
 $Comp
-L GND #PWR16
+L GND #PWR023
 U 1 1 552837AD
 P 7800 1200
-F 0 "#PWR16" H 7800 1200 30  0001 C CNN
+F 0 "#PWR023" H 7800 1200 30  0001 C CNN
 F 1 "GND" H 7800 1130 30  0001 C CNN
 F 2 "" H 7800 1200 60  0000 C CNN
@@
 $EndComp
 $Comp
-L GND #PWR19
+L GND #PWR024
 U 1 1 5530A16F
 P 8350 6200
-F 0 "#PWR19" H 8350 6200 30  0001 C CNN
+F 0 "#PWR024" H 8350 6200 30  0001 C CNN
 F 1 "GND" H 8350 6130 30  0001 C CNN
 F 2 "" H 8350 6200 60  0000 C CNN
@@
 	7800 6200 7650 6200
 Wire Wire Line
-	9500 1900 10250 1900
+	9350 1950 10650 1950
 Wire Wire Line
 	10200 6400 9900 6400
@@
 $EndComp
 $Comp
-L GND #PWR10
+L GND #PWR025
 U 1 1 5539BEBB
 P 3900 4050
-F 0 "#PWR10" H 3900 4050 30  0001 C CNN
+F 0 "#PWR025" H 3900 4050 30  0001 C CNN
 F 1 "GND" H 3900 3980 30  0001 C CNN
 F 2 "" H 3900 4050 60  0000 C CNN
@@
 	2200 3850 2650 3850
 $Comp
-L C C?
+L C C8
 U 1 1 5542E5DC
 P 2200 4050
-F 0 "C?" H 2200 4150 40  0000 L CNN
+F 0 "C8" H 2200 4150 40  0000 L CNN
 F 1 "4.7 uF" H 2206 3965 40  0000 L CNN
 F 2 "~" H 2238 3900 30  0000 C CNN
@@
 	1    0    0    -1
 $EndComp
-Wire Notes Line
-	9450 1350 9450 2100
-Wire Notes Line
-	9450 2100 10900 2100
-Wire Notes Line
-	10900 2100 10900 1000
-Wire Notes Line
-	10900 1000 9600 1000
 Wire Wire Line
 	2600 3850 2600 3950
 $Comp
-L GND #PWR?
+L GND #PWR026
 U 1 1 55430D54
 P 2200 4300
-F 0 "#PWR?" H 2200 4300 30  0001 C CNN
+F 0 "#PWR026" H 2200 4300 30  0001 C CNN
 F 1 "GND" H 2200 4230 30  0001 C CNN
 F 2 "" H 2200 4300 60  0000 C CNN
@@
 	2200 4300 2200 4250
 $Comp
-L NPN Q?
+L NPN Q3
 U 1 1 554310E6
-P 9900 1300
-F 0 "Q?" H 9900 1150 50  0000 R CNN
-F 1 "NPN" H 9900 1450 50  0000 R CNN
-F 2 "~" H 9900 1300 60  0000 C CNN
-F 3 "~" H 9900 1300 60  0000 C CNN
-	1    9900 1300
-	0    1    1    0
-$EndComp
-$Comp
-L NPN Q?
+P 10000 1650
+F 0 "Q3" H 10000 1500 50  0000 R CNN
+F 1 "NPN" H 10000 1800 50  0000 R CNN
+F 2 "~" H 10000 1650 60  0000 C CNN
+F 3 "~" H 10000 1650 60  0000 C CNN
+	1    10000 1650
+	0    1    1    0
+$EndComp
+$Comp
+L NPN Q4
 U 1 1 554310F6
-P 10100 1700
-F 0 "Q?" H 10100 1550 50  0000 R CNN
-F 1 "NPN" H 10100 1850 50  0000 R CNN
-F 2 "~" H 10100 1700 60  0000 C CNN
-F 3 "~" H 10100 1700 60  0000 C CNN
-	1    10100 1700
-	0    1    1    0
-$EndComp
-$Comp
-L NPN Q?
+P 10450 1750
+F 0 "Q4" H 10450 1600 50  0000 R CNN
+F 1 "NPN" H 10450 1900 50  0000 R CNN
+F 2 "~" H 10450 1750 60  0000 C CNN
+F 3 "~" H 10450 1750 60  0000 C CNN
+	1    10450 1750
+	0    1    1    0
+$EndComp
+$Comp
+L NPN Q2
 U 1 1 554310FC
-P 9250 1250
-F 0 "Q?" H 9250 1100 50  0000 R CNN
-F 1 "NPN" H 9250 1400 50  0000 R CNN
-F 2 "~" H 9250 1250 60  0000 C CNN
-F 3 "~" H 9250 1250 60  0000 C CNN
-	1    9250 1250
-	0    1    1    0
-$EndComp
+P 9550 1550
+F 0 "Q2" H 9550 1400 50  0000 R CNN
+F 1 "NPN" H 9550 1700 50  0000 R CNN
+F 2 "~" H 9550 1550 60  0000 C CNN
+F 3 "~" H 9550 1550 60  0000 C CNN
+	1    9550 1550
+	0    1    1    0
+$EndComp
+Text GLabel 10700 1000 2    60   Input ~ 0
+VBatt
+Wire Wire Line
+	9750 1650 9750 1000
+Wire Wire Line
+	9750 1000 10700 1000
+Wire Wire Line
+	10200 1750 10200 1000
+Connection ~ 10200 1000
+Wire Wire Line
+	10650 1850 10650 1000
+Connection ~ 10650 1000
+Wire Wire Line
+	9800 1750 9350 1750
+Wire Wire Line
+	10250 1850 9350 1850
 $EndSCHEMATC
