File: KiCad/Player-Health/Player-Health.kicad_pcb (KiCad board)
At the start: 2 copper layers, 98 x 64.9 mm, 34 parts, among them IC1 ATMEGA328-P, J1 MICRO_USB, M1 RUMBLE, P1 2P_CGRID_M, P2 6pM CGrid, P3 6pM Header, P4 8pF Header, Q1 NPN, U1 MCP73831, U2 LM1084IT-3.3/NOPB, U3 14SLED, U4 ESP8266, X1 CRYSTAL

Commit message: Quick Update #4 4/24
Other:
- board text added: "400 mAh LiPo"
Changed lines of the file:
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@@
     (area 39.104712 86.614799 138.459601 152.1206)
     (thickness 1.6)
-    (drawings 23)
+    (drawings 24)
     (tracks 186)
     (zones 0)
@@
     )
   )
+  (gr_text "400 mAh LiPo" (at 59.1058 131.4958) (layer F.SilkS)
+    (effects (font (size 2 2) (thickness 0.3)))
+  )
   (gr_line (start 138.4046 86.6648) (end 43.3832 86.6648) (angle 90) (layer Edge.Cuts) (width 0.1))

Commit message: Quick Update #5 4/24
Routing:
- net +3.3V: track 53.2 -> 8.94 mm, vias 3 -> 1
Changed lines of the file:
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@@
     (thickness 1.6)
     (drawings 24)
-    (tracks 186)
+    (tracks 178)
     (zones 0)
     (modules 34)
@@
     (effects (font (size 1.5 1.5) (thickness 0.3)))
   )
-  (segment (start 87.7824 100.7364) (end 87.7824 96.98482) (width 0.508) (layer F.Cu) (net 1))
-  (segment (start 87.7824 96.98482) (end 86.42858 95.631) (width 0.508) (layer F.Cu) (net 1))
-  (segment (start 65.3034 107.5182) (end 69.5198 107.5182) (width 0.508) (layer F.Cu) (net 1))
-  (segment (start 69.5198 107.5182) (end 71.6534 105.3846) (width 0.508) (layer F.Cu) (net 1))
-  (segment (start 91.6432 110.744) (end 91.6432 104.5972) (width 0.508) (layer F.Cu) (net 1))
-  (segment (start 83.1342 105.3846) (end 71.6534 105.3846) (width 0.508) (layer F.Cu) (net 1))
-  (segment (start 87.7824 100.7364) (end 83.1342 105.3846) (width 0.508) (layer F.Cu) (net 1))
-  (via (at 87.7824 100.7364) (size 0.889) (layers F.Cu B.Cu) (net 1))
-  (segment (start 91.6432 104.5972) (end 87.7824 100.7364) (width 0.508) (layer B.Cu) (net 1))
-  (via (at 91.6432 104.5972) (size 0.889) (layers F.Cu B.Cu) (net 1))
+  (segment (start 86.42858 95.631) (end 84.6836 95.631) (width 0.508) (layer F.Cu) (net 1) (status 400000))
+  (segment (start 84.709 95.6564) (end 84.709 95.6818) (width 0.508) (layer B.Cu) (net 1))
+  (segment (start 84.6836 95.631) (end 84.709 95.6564) (width 0.508) (layer B.Cu) (net 1))
+  (via (at 84.6836 95.631) (size 0.889) (layers F.Cu B.Cu) (net 1))
   (segment (start 91.6432 110.744) (end 94.3102 110.744) (width 0.508) (layer B.Cu) (net 1))
   (segment (start 94.3102 110.744) (end 94.361 110.6932) (width 0.508) (layer B.Cu) (net 1))
   (segment (start 59.1312 110.8202) (end 59.1312 110.1598) (width 0.508) (layer B.Cu) (net 1))
   (segment (start 59.1312 110.1598) (end 61.7728 107.5182) (width 0.508) (layer B.Cu) (net 1))
-  (segment (start 61.7728 107.5182) (end 65.3034 107.5182) (width 0.508) (layer B.Cu) (net 1))
-  (via (at 65.3034 107.5182) (size 0.889) (layers F.Cu B.Cu) (net 1))
   (segment (start 59.1312 115.9002) (end 54.2544 115.9002) (width 0.508) (layer B.Cu) (net 2) (status 400000))
   (segment (start 52.451 114.0968) (end 52.451 109.9312) (width 0.508) (layer B.Cu) (net 2) (status 800000))
