File: KiCad/Player-Health/Player-Health.kicad_pcb (KiCad board)
At the start: 2 copper layers, 98 x 64.9 mm, 34 parts, among them IC1 ATMEGA328-P, J1 MICRO_USB, M1 RUMBLE, P1 2P_CGRID_M, P2 6pM CGrid, P3 6pM Header, P4 8pF Header, Q1 NPN, U1 MCP73831, U2 LM1084IT-3.3/NOPB, U3 14SLED, U4 ESP8266, X1 CRYSTAL

Commit message: Quick Update #3 5/1
Potential last changes before ordering ir receiver and player boards
Parts:
- added C8: 4.7 uF, C2, F.Cu at (104.9, 104.5)
- added Q2: NPN, TO92, F.Cu at (107.7, 144.5)
- added Q3: NPN, TO92, F.Cu at (100.7, 144.3)
- added Q4: NPN, TO92, F.Cu at (93.6, 144.1)
- moved U4 5.26 mm to (87.5, 133.8)
- moved P2 5.26 mm to (91.2, 149.8)
- moved IC1 5.11 mm to (98.9, 106.9)
- moved P4 3.75 mm to (127.7, 140.6)
- moved D3 2.25 mm to (85.3, 95.2)
- moved JP2 1.83 mm to (83.5, 142.7)
Connections:
- P2 pad 4: LED G -> N-0000023
- P2 pad 5: LED B -> N-0000024
- P2 pad 6: LED R -> N-0000025
- R3 pad 1: (no net) -> VSense
Routing:
- net VBatt: track 172.4 -> 211.5 mm
- net GND: track 27.6 -> 61.0 mm, vias 0 -> 1
- net +3.3V: track 8.94 -> 31.4 mm, vias 1 -> 2
- net N-0000025: track 0.00 -> 10.6 mm
- net IR Sense: track 20.9 -> 28.6 mm
- net Reset: track 43.6 -> 50.1 mm, vias 0 -> 1
- net I2C CLK: track 27.8 -> 34.2 mm, vias 1 -> 0
- net N-0000024: track 0.00 -> 6.23 mm
- net UART TX: track 43.6 -> 37.9 mm
- net UART RX: track 65.9 -> 60.9 mm, vias 1 -> 0
- net Rumble: track 32.3 -> 37.2 mm
- net N-0000023: track 0.00 -> 4.52 mm
- net N-0000020: track 2.26 -> 6.32 mm
- net MOSI: track 32.0 -> 35.6 mm
- net MISO: track 35.6 -> 39.1 mm
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