File: KiCad/IR-Reciever/IR-RecieverV2.kicad_pcb (KiCad board)
At the start: 2 copper layers, 19.7 x 27.8 mm, 6 parts, among them P1 CONN_6, U1 TSOP38238, U2 TSOP38238, U3 TSOP38238, U4 RGBLED

Commit message: Ordered Weapon Proto
Tada... Holy Crap
Routing:
- net N-000001: track 30.9 -> 28.8 mm
Changed lines of the file:
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@@
     (thickness 1.6)
     (drawings 22)
-    (tracks 21)
+    (tracks 22)
     (zones 0)
     (modules 6)
@@
   (segment (start 39.37 33.02) (end 38.1 34.29) (width 0.254) (layer F.Cu) (net 1))
   (segment (start 39.37 30.48) (end 39.37 33.02) (width 0.254) (layer F.Cu) (net 1))
-  (segment (start 35.56 35.56) (end 38.1 35.56) (width 0.254) (layer B.Cu) (net 2))
+  (segment (start 40.005 33.655) (end 36.5506 33.655) (width 0.254) (layer B.Cu) (net 2))
+  (segment (start 36.5506 33.655) (end 35.56 32.6644) (width 0.254) (layer B.Cu) (net 2))
+  (segment (start 31.115 32.385) (end 32.9946 32.385) (width 0.254) (layer B.Cu) (net 2))
+  (segment (start 32.9946 32.385) (end 35.56 29.8196) (width 0.254) (layer B.Cu) (net 2))
   (segment (start 40.005 33.655) (end 43.815 33.655) (width 0.254) (layer B.Cu) (net 2))
-  (segment (start 38.1 35.56) (end 40.005 33.655) (width 0.254) (layer B.Cu) (net 2))
-  (segment (start 35.56 35.56) (end 35.56 24.765) (width 0.254) (layer B.Cu) (net 2))
+  (segment (start 35.56 35.56) (end 35.56 32.6644) (width 0.254) (layer B.Cu) (net 2))
+  (segment (start 35.56 32.6644) (end 35.56 29.8196) (width 0.254) (layer B.Cu) (net 2))
+  (segment (start 35.56 29.8196) (end 35.56 24.765) (width 0.254) (layer B.Cu) (net 2))
   (segment (start 29.21 32.385) (end 31.115 32.385) (width 0.254) (layer B.Cu) (net 2))
   (segment (start 35.56 35.56) (end 35.56 37.465) (width 0.254) (layer B.Cu) (net 2))
-  (segment (start 31.75 35.56) (end 35.56 35.56) (width 0.254) (layer B.Cu) (net 2))
-  (segment (start 31.75 33.02) (end 31.75 35.56) (width 0.254) (layer B.Cu) (net 2))
-  (segment (start 31.115 32.385) (end 31.75 33.02) (width 0.254) (layer B.Cu) (net 2))
   (segment (start 36.83 30.48) (end 29.845 30.48) (width 0.254) (layer F.Cu) (net 3))
   (segment (start 29.845 30.48) (end 29.21 29.845) (width 0.254) (layer F.Cu) (net 3))
